File: device/hw/$pr/south_bridge.kicad_sch (KiCad schematic)
At the start: 0 parts

Commit message: Add sheets
Other:
- removed sheet North Bridge
- removed sheet South Bridge
- added sheet Battery Managment System (bms.kicad_sch)
- added sheet STM32 MCU (stm32_mcu.kicad_sch)
Changed lines of the file:
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@@
 	(paper "A4")
 	(sheet
-		(at 43.18 50.8)
-		(size 35.56 26.67)
+		(at 64.77 54.61)
+		(size 31.75 22.86)
 		(fields_autoplaced yes)
 		(stroke
@@
 			(color 0 0 0 0.0000)
 		)
-		(property "Sheetname" "South Bridge"
-			(at 43.18 50.0884 0)
+		(property "Sheetname" "Battery Managment System"
+			(at 64.77 53.8984 0)
 			(effects
 				(font
@@
 			)
 		)
-		(property "Sheetfile" "south_bridge.kicad_sch"
-			(at 43.18 78.0546 0)
+		(property "Sheetfile" "bms.kicad_sch"
+			(at 64.77 78.0546 0)
 			(effects
 				(font
@@
 		(instances
 			(project "medmentum"
-				(path "/ead52261-b3da-41ef-908f-3daaabe10954"
-					(page "2")
+				(path "/ead52261-b3da-41ef-908f-3daaabe10954/940ef1bd-73e9-475b-b1ba-056ab9b45d18"
+					(page "3")
 				)
 			)
@@
 	)
 	(sheet
-		(at 153.67 52.07)
-		(size 34.29 21.59)
+		(at 129.54 54.61)
+		(size 31.75 24.13)
 		(fields_autoplaced yes)
 		(stroke
@@
 			(color 0 0 0 0.0000)
 		)
-		(property "Sheetname" "North Bridge"
-			(at 153.67 51.3584 0)
+		(property "Sheetname" "STM32 MCU"
+			(at 129.54 53.8984 0)
 			(effects
 				(font
@@
 			)
 		)
-		(property "Sheetfile" "north_bridge.kicad_sch"
-			(at 153.67 74.2446 0)
+		(property "Sheetfile" "stm32_mcu.kicad_sch"
+			(at 129.54 79.3246 0)
 			(effects
 				(font
@@
 		(instances
 			(project "medmentum"
-				(path "/ead52261-b3da-41ef-908f-3daaabe10954"
-					(page "5")
+				(path "/ead52261-b3da-41ef-908f-3daaabe10954/940ef1bd-73e9-475b-b1ba-056ab9b45d18"
+					(page "4")
 				)
 			)
 		)
 	)
-	(sheet_instances
-		(path "/"
-			(page "1")
-		)
-	)
