File: device/hw/$pr/medmentum.kicad_sch (KiCad schematic)
At the start: 0 parts

Commit message: Sheets
Other:
- added sheet Peripherals (Sheets/peripherals.kicad_sch)
Changed lines of the file:
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@@
+		)
+	)
+	(sheet
+		(at 99.06 78.74)
+		(size 27.94 22.86)
+		(fields_autoplaced yes)
+		(stroke
+			(width 0.1524)
+			(type solid)
+		)
+		(fill
+			(color 0 0 0 0.0000)
+		)
+		(property "Sheetname" "Peripherals"
+			(at 99.06 78.0284 0)
+			(effects
+				(font
+					(size 1.27 1.27)
+				)
+				(justify left bottom)
+			)
+		)
+		(property "Sheetfile" "Sheets/peripherals.kicad_sch"
+			(at 99.06 102.1846 0)
+			(effects
+				(font
+					(size 1.27 1.27)
+				)
+				(justify left top)
+			)
+		)
+		(instances
+			(project "medmentum"
+				(path "/ead52261-b3da-41ef-908f-3daaabe10954"
+					(page "7")
+				)
+			)
 		)
 	)

Commit message: BMS
Other:
- company: (none) -> ETŠ Mihajlo Pupin "Medmentum"
Changed lines of the file:
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@@
 	(generator_version "8.0")
 	(paper "A4")
+	(title_block
+		(company "ETŠ Mihajlo Pupin \"Medmentum\"")
+	)
 	(sheet
 		(at 43.18 50.8)

Commit message: application
Parts:
- added BAT1: 2000mAh, fpl:BAT-TH_BH-18650-A5BJ003, symbol Device:Battery_Cell
- added BZ3: Buzzer, symbol Device:Buzzer
- added C1: 100n, Capacitor_SMD:C_0603_1608Metric, symbol Device:C_Small
- added C10, C3, C4, C5, C53, C57, C58, C59, C60, C61, C62, C65, C72: 100n, Capacitor_SMD:C_0603_1608Metric, symbol Device:C
- added C11, C55, C70, C71, C9: 1u, Capacitor_SMD:C_0603_1608Metric, symbol Device:C
- added C2, C54, C56, C63, C64, C73: 4.7u, Capacitor_SMD:C_0805_2012Metric, symbol Device:C
- added C6, C7, C74, C8: 10u, Capacitor_SMD:C_0805_2012Metric, symbol Device:C
- added C66, C67: 5p, Capacitor_SMD:C_0402_1005Metric, symbol Device:C
- added C68, C69: 16p, Capacitor_SMD:C_0402_1005Metric, symbol Device:C
- added C75: 22u, Capacitor_SMD:C_0805_2012Metric, symbol Device:C
- added CON3: ZX-IDC2.54-2-13PZZ, fpl:IDC-TH_26P-P2.54_ZX-IDC2.54-2-13PZZ, symbol syl:ZX-IDC2.54-2-13PZZ
- added D1, D17, D18, D19, D2, D20, D3, D4, D5: LED, LED_SMD:LED_0603_1608Metric, symbol Device:LED
- added FB2: 100R@100MHz, Inductor_SMD:L_0805_2012Metric, symbol Device:FerriteBead
- added L1: 2.2u, Inductor_SMD:L_1008_2520Metric, symbol Device:L
- added L2: 1u, Capacitor_SMD:C_0603_1608Metric, symbol Device:L
- added Q5: PNP, symbol Simulation_SPICE:PNP
- added Q6, Q7: NPN, Package_TO_SOT_SMD:SOT-23, symbol Simulation_SPICE:NPN
- added R1, R11, R20, R9, R94, R95: 10k, Resistor_SMD:R_0402_1005Metric, symbol Device:R
- added R10, R14, R17, R18: 0, Resistor_SMD:R_0805_2012Metric, symbol Device:R_Small
- added R100, R13, R15, R16, R2, R90, R92, R93, R97, R98, R99: 47, symbol Device:R_Small
- added R12, R3, R8: 10k, Resistor_SMD:R_0402_1005Metric, symbol Device:R_Small
- added R19: 1.2K, Resistor_SMD:R_0603_1608Metric, symbol Device:R
- added R21, R7: 220, symbol Device:R_Small
- added R22: 2.7K, Resistor_SMD:R_0603_1608Metric, symbol Device:R
- added R23, R24, R82, R83, R85, R86, R87: 5.1k, Resistor_SMD:R_0402_1005Metric, symbol Device:R_Small
- added R4: 100, Resistor_SMD:R_0603_1608Metric, symbol Device:R
- added R5, R6: 5.1k 1%, Resistor_SMD:R_0402_1005Metric, symbol Device:R
- added R79: 820, Resistor_SMD:R_0603_1608Metric, symbol Device:R
- added R80, R81: 100k, Resistor_SMD:R_0603_1608Metric, symbol Device:R_Small
- added R84, R88: 1k, symbol Device:R_Small
- added R89, R96: 1k, Resistor_SMD:R_2512_6332Metric, symbol Device:R_Small
- added R91: 10m 1% 1W, Resistor_SMD:R_1206_3216Metric, symbol Device:R
- added SW1, SW11, SW9: SW_SPDT, symbol Switch:SW_SPDT
- added SW10, SW12: SW_Push, symbol Switch:SW_Push
- added TH1: 10K, symbol Device:Thermistor_NTC
- added U1: TS3USB221ARSER, fpl:TS3USB221ARSER, symbol syl:TS3USB221ARSER
- added U16: BQ27441DRZR-G1B, fpl:BQ27441DRZR-G1B, symbol syl:BQ27441DRZR-G1B
- added U17: TPS62082DSGR, fpl:TPS62082DSGR, symbol syl:TPS62082DSGR
- added U2: TPS63002DRCT, fpl:TPS63002DRCR, symbol syl:TPS63002DRCT
- added U3: USBLC6-2SC6, fpl:USBLC6-2SC6, symbol syl:USBLC6-2SC6
- added U4: ESP32-C3-MINI-1-H4, fpl:ESP32-C3-MINI-1-H4, symbol syl:ESP32-C3-MINI-1-H4(4MB)
- added U5: BQ24074RGTR, fpl:BQ24074RGTR, symbol syl:BQ24074RGTR
- added U6: STM32F411CEU6, fpl:STM32F411CEU6, symbol syl:STM32F411CEU6
- added USB1: USB-310F-B-SU, fpl:USB-310F-B-SU, symbol syl:USB-310F-B-SU
- added Y3: 12.5pF, Crystal:Crystal_SMD_3215-2Pin_3.2x1.5mm, symbol Device:Crystal_Small
- added Y4: 18pF, Crystal:Crystal_SMD_3225-4Pin_3.2x2.5mm, symbol Device:Crystal_GND24_Small
Connections:
- new net: U1.8 (D+), U3.4
- new net: U1.7 (D-), U3.6
- new net: C11.2, R8.2, U4.5 (IO2)
- new net: D2.2 (A), R2.1
- new net: D19.1 (K), R97.2
- new net: D3.1 (K), R13.1
- new net: D3.2 (A), D5.1 (K), R9.1, SW1.2 (B)
- new net: Q5.2 (B), R84.2
- new net: D18.2 (A), R93.1
- new net: D5.2 (A), R16.1
- new net: R16.2, R17.1
- new net: D4.1 (K), R15.2
- new net: R11.2, U4.23 (IO9)
- new net: R12.1, U4.22 (IO8)
- new net: C73.2, U6.22 (VCAP_1)
- new net: R10.1, R9.2
- new net: L2.1, U17.7 (SW)
- new net: R3.2, U1.6 (~{OE})
- new net: U4.10 (NC), U4.15 (NC), U4.17 (NC), U4.24 (NC), U4.25 (NC), U4.28 (NC), U4.29 (NC), U4.32 (NC), U4.33 (NC), U4.34 (NC), U4.35 (NC), U4.4 (NC), U4.7 (NC), U4.9 (NC)
- new net: L1.2, U2.2 (L2)
- new net: L1.1, U2.4 (L1)
- new net: R13.2, R14.1
- new net: Q7.2 (B), R96.1
- new net: R84.1, U6.37 (PA14)
- new net: Q6.2 (B), R88.2
- new net: R98.1, U6.13 (PA3)
- new net: D1.1 (K), R7.2
- new net: BZ3.2 (-), Q7.1 (C), R89.1
- new net: R20.2, U5.4 (~{CE})
- new net: D17.1 (K), R21.2
- new net: C70.1, U16.5 (VDD)
- new net: R99.2, U6.12 (PA2)
- new net: D20.1 (K), R100.2
- new net +USB_D: U3.3, USB1.10 (D+), USB1.8 (D+)
- new net +USB_DESP: U1.3 (2D+), U4.27 (IO19)
- new net +USB_DSTM: U1.1 (1D+), U6.33 (PA12)
- new net -USB_D: U3.1, USB1.7 (D-), USB1.9 (D-)
- new net -USB_DESP: U1.4 (2D-), U4.26 (IO18)
- new net -USB_DSTM: U1.2 (1D-), U6.32 (PA11)
- new net BAT: BAT1.1 (+), C71.2, R91.2, U16.6 (BAT), U16.8 (SRP)
- new net BATSYS: R91.1, U16.7 (SRN), U5.2 (BAT), U5.3 (BAT)
- new net BCK5_EN: C10.2, R4.1, U2.6 (EN), U2.7 (PS/SYNC), U2.8 (VINA)
- new net BCKOUT33: C1.2, C2.1, C3.1, C4.1, C5.1, C63.2, C75.2, CON3.20, CON3.21, CON3.24, CON3.25, D20.2 (A), FB2.1, L2.2, Q5.3 (E), R1.2, R12.2, R18.1, R8.1, R80.1, R81.1, R85.2, R86.2, R87.2, SW1.3 (C), SW11.3 (C), SW9.3 (C), U1.10 (VCC), U17.5 (VOS), U4.3 (3V3)
- new net BCKOUT5: C7.2, C74.2, C8.2, CON3.12, CON3.13, CON3.2, CON3.4, D1.2 (A), U17.1 (EN), U17.8 (VIN), U2.1 (VOUT), U2.10 (FB)
- new net BCOUT: C54.2, C6.2, R4.2, U2.5 (VIN), U5.10 (OUT), U5.5 (EN2)
- new net BOOT0: R95.2, U6.44 (BOOT0)
- new net BUZPWM: R96.2, U6.29 (PA8)
- new net BUZVCC: BZ3.1 (+), R89.2
- new net CC1: R5.1, USB1.6 (CC1)
- new net CC2: R6.1, USB1.12 (CC2)
- new net CHG_#CHG: R80.2, U5.9 (~{CHG}), U6.28 (PB15)
- new net CHG_#PGOOD: R81.2, U5.7 (~{PGOOD}), U6.27 (PB14)
- new net CONFSW: CON3.22, U6.41 (PB5)
- new net DISPEN: U6.34 (PA13)
- new net ENRST: C53.1, C9.1, R1.1, SW10.1, U4.8 (EN)
- new net FG_BIN: R94.1, U16.10 (BIN)
- new net FG_GPOUT: R87.1, U16.12 (GPOUT), U6.26 (PB13)
- new net FG_SCL: R23.2, R85.1, U16.2 (SCL), U6.21 (PB10)
- new net FG_SDA: R83.2, R86.1, U16.1 (SDA), U6.39 (PB3)
- new net GND: BAT1.2 (-), C1.1, C10.1, C11.1, C2.2, C3.2, C4.2, C5.2, C53.2, C54.1, C55.2, C56.1, C57.1, C58.1, C59.1, C6.1, C60.1, C61.1, C62.1, C66.2, C67.1, C68.2, C69.1, C7.1, C70.2, C71.1, C72.1, C73.1, C74.1, C75.1, C8.1, C9.2, CON3.14, CON3.15, CON3.6, CON3.8, Q6.3 (E), Q7.3 (E), R19.1, R20.1, R21.1, R22.1, R23.1, R24.2, R3.1, R5.2, R6.2, R7.1, R79.1, R82.1, R83.1, R94.2, SW1.1 (A), SW10.2, SW11.1 (A), SW12.1, SW9.1 (A), TH1.2, U1.5 (GND), U16.13 (EXP), U16.3 (VSS), U17.2 (GND), U17.3 (MODE), U17.9 (GND), U17.9_1 (GND), U17.9_2 (GND), U2.11 (PP), U2.3 (PGND), U2.9 (GND), U3.2, U4.1 (GND), U4.11 (GND), U4.14 (GND), U4.2 (GND), U4.36 (GND), U4.37 (GND), U4.38 (GND), U4.39 (GND), U4.40 (GND), U4.41 (GND), U4.42 (GND), U4.43 (GND), U4.44 (GND), U4.45 (GND), U4.46 (GND), U4.47 (GND), U4.48 (GND), U4.49 (GND), U4.50 (GND), U4.51 (GND), U4.52 (GND), U4.53 (GND), U5.14 (TMR), U5.17 (EXP), U5.6 (EN1), U5.8 (VSS), U6.23 (VSS), U6.35 (VSS), U6.47 (VSS), U6.49 (VSS), USB1.1 (GND), USB1.15 (GND), USB1.16 (GND), USB1.2 (GND), Y4.2, Y4.4
- new net GNDA: C63.1, C64.1, C65.1, U6.8 (VSSA)
- new net HOSW: CON3.26, U6.45 (PB8)
- new net HSE_IN: C68.1, U6.5 (PH0-OSC_IN), Y4.1
- new net HSE_OUT: C69.2, U6.6 (PH1-OSC_OUT), Y4.3
- new net IICDISP_SCL: CON3.9, R82.2, U6.42 (PB6)
- new net IICDISP_SDA: CON3.11, R24.1, U6.43 (PB7)
- new net ILIM: R19.2, U5.12 (ILIM)
- new net ISET: R79.2, U5.16 (ISET)
- new net ITERM: R22.2, U5.15 (ITERM)
- new net LEDCHPWM: CON3.19, R99.1
- new net LEDHOPWM: CON3.23, R98.2
- new net LGND: Q6.1 (C), R100.1, R14.2, R15.1, R97.1
- new net LSE_IN: C66.1, U6.3 (PC14-OSC32_IN), Y3.2
- new net LSE_OUT: C67.2, U6.4 (PC15-OSC32_OUT), Y3.1
- new net LVCC: Q5.1 (C), R17.2, R2.2, R88.1, R93.2
- new net NRST: C72.2, SW12.2, U6.7 (NRST)
- new net PANICGPIO: CON3.17, U6.25 (PB12)
- new net PANICPWM1: CON3.18, U6.11 (PA1)
- new net PANICPWM2: CON3.16
- new net SERVOPWM1: CON3.1, U6.16 (PA6)
- new net SERVOPWM2: CON3.3, U6.17 (PA7)
- new net SERVOPWM3: CON3.5, U6.18 (PB0)
- new net SERVOPWM4: CON3.7, U6.19 (PB1)
- new net SERVOPWM5: CON3.10, U6.10 (PA0-WKUP)
- new net STM_UARTRX: R90.1, U6.31 (PA10)
- new net STM_UARTTX: R92.1, U6.30 (PA9)
- new net SW_BOOT0: D18.1 (K), D19.2 (A), D2.1 (K), D4.2 (A), R11.1, R95.1, SW11.2 (B), SW9.2 (B)
- new net TS: TH1.1, U5.1 (TS)
- new net UARTRX_ESP: R90.2, U4.31 (TXD0)
- new net UARTTX_ESP: R92.2, U4.30 (RXD0)
- new net USB_SLC: R10.2, U1.9 (S)
- new net VBUS: C55.1, D17.2 (A), U3.5, U5.13 (IN), USB1.13 (VBUS), USB1.14 (VBUS), USB1.3 (VBUS), USB1.4 (VBUS)
- new net VDD: C56.2, C57.2, C58.2, C59.2, C60.2, C61.2, C62.2, R18.2, U6.1 (VBAT), U6.24 (VDD), U6.36 (VDD), U6.48 (VDD)
- new net VDDASTM: C64.2, C65.2, FB2.2, U6.9 (VREF+)
- no-connect marks 0 -> 17
Other:
- removed sheet North Bridge
- removed sheet Peripherals
- removed sheet South Bridge
- note added: "1."
- note added: "2."
- note added: "3."
- note added: "4."
- note added: "5."
- note added: "6."
- note added: "7."
- note added: "8."
- note added: "Battery Charging IC"
- note added: "Battery Fuel Gauge IC"
- note added: "Birač za USB Input Source"
- note added: "Boot memory picker."
- note added: "Buck-Boost Fixed 3.3V Converter"
- note added: "Buck-Boost Fixed 5V Converter"
- note added: "ESP32-C3 MINI 1"
- note added: "GPIO9 SPI 1 GPIO9 Joint Download Boot USB 0"
- note added: "HSE (High Speed External) Clock."
- note added: "IIC "Pull-up" otpornici."
- note added: "LED Debug mode picker."
- note added: "LSE (Low Speed External) Clock."
- note added: "Reset."
- note added: "STM32F411CE MCU"
- note added: "TIM1"
- note added: "TIM2"
- note added: "TIM3"
- note added: "USB-C Connector"
- note added: "USB-C Konektor, [USBLC6-2SC6] TVS Diode Protection i [TS3USB221ARSER] 1:2 Multiplexer za USB Host"
- note added: "[BQ24074RGTR] IC za punjenje i pražnjenje baterije."
- note added: "[BQ27441DRZR-G1B] IC za praćenje stanja baterije i [BAT1 (SAMSUNG20R)] 2000mAh baterija."
- note added: "[TPS62082DSGR] Fiksni 3.3V Step-Down konverter BCKOUT5(TPS63002DRCT)-->BCKOUT33(TPS62082DSGR)"
- note added: "[TPS63002DRCT] Fiksni 5V Boost konverter BCOUT(BQ24074RGTR)-->BCKOUT5(TPS63002DRCT)"
- note added: "Čišćenje signala od šuma za analogno napajanje."
- note added: "Čišćenje signala od šuma za digitalno napajanje."

Commit message: application
Parts:
- removed R11: 10k, Resistor_SMD:R_0402_1005Metric, symbol Device:R
- added C12, C13: 100n, symbol Device:C_Small
- added R11: 10k, symbol Device:R_Small
- added R25: 0, symbol Device:R_Small
- added R26, R29: 1k, Resistor_SMD:R_2512_6332Metric, symbol Device:R_Small
- added R27, R28: 10k, Resistor_SMD:R_2512_6332Metric, symbol Device:R_Small
- BZ3: footprint (none) -> fpl:BUZ-TH_BD17.0-P10.00-D0.8
- R96: value 1k -> 47
- renumbered CON3 to CON
Connections:
- net BUZVCC is gone; now on net BCKOUT5: BZ3.1 (+), R89.2
- net BCKOUT33: now also CON.19, R27.1, R28.1; no longer CON.20, CON.24, CON.25
- net BCKOUT5: now also CON.23, CON.5, CON.7; no longer CON.13, CON.2, CON.4
- net CONFSW: now also C12.1, R26.1, R27.2; no longer CON.22
- net GND: now also CON.13, CON.17, CON.24, C12.2, C13.2; no longer CON.14
- net HOSW: now also C13.1, R28.2, R29.1; no longer CON.26
- net IICDISP_SDA: now also CON.10; no longer CON.11
- net LEDCHPWM: now also CON.18; no longer CON.19
- net LEDHOPWM: now also CON.20; no longer CON.23
- net PANICGPIO: now also CON.26; no longer CON.17
- net SERVOPWM2: now also CON.2; no longer CON.3
- net SERVOPWM3: now also CON.3; no longer CON.5
- net SERVOPWM4: now also CON.4; no longer CON.7
- net SERVOPWM5: now also CON.11; no longer CON.10
- net SW_BOOT0: now also R11.1
- net at U4.23 (IO9): now also R25.2
- net PANICPWM: now reaches U6.46 (PB9)
- net PANICPWM: now also CON.25
- net DISPEN: no longer names the net of U6.34 (PA13)
- net PANICPWM1 renamed SERVOPWM6
- net SERVOPWM6: now also CON.22; no longer CON.18
- net PANICPWM2 renamed HOSW_DB
- net HOSW_DB: now also R29.2
- new net: R11.2, R25.1
- new net CONFSW_DB: CON.14, R26.2
- no-connect marks 17 -> 19
Other:
- note added: "PWM Buzzer Driver"
- note added: "South Bus IDC"
- note added: "Switch Debounce Suppressor"
- note added: "TIM4"
- note removed: "GPIO9 SPI 1 GPIO9 Joint Download Boot USB 0"
- company: ETŠ Mihajlo Pupin "Medmentum" -> ETŠ Mihajlo Pupin "Medmentum" - Guteša Ognjen T31
- title: (none) -> Medmentum 
- moved on the sheet: BZ3, CON, D4, Q7, R15, R23, R24, R82, R83, R89, R96

Commit message: application
Parts:
- removed R14, R17: 0, Resistor_SMD:R_0805_2012Metric, symbol Device:R_Small
- removed R4: 100, Resistor_SMD:R_0603_1608Metric, symbol Device:R
- added R20: 0, Resistor_SMD:R_0805_2012Metric, symbol Device:R_Small
- added R21, R25: 47, Resistor_SMD:R_0603_1608Metric, symbol Device:R_Small
- BZ1: renamed from BZ3; LCSCPart (none) -> C76872
- C35: renamed from C13; footprint (none) -> Capacitor_SMD:C_0603_1608Metric; LCSCPart (none) -> C14663
- C36: renamed from C12; footprint (none) -> Capacitor_SMD:C_0603_1608Metric; LCSCPart (none) -> C14663
- D1: renamed from D17; footprint LED_SMD:LED_0603_1608Metric -> LED_SMD:LED_0805_2012Metric; LCSCPart C2290 -> C2297
- D4: renamed from D20; footprint LED_SMD:LED_0603_1608Metric -> LED_SMD:LED_0805_2012Metric; LCSCPart C2290 -> C2297
- D7: renamed from D1; footprint LED_SMD:LED_0603_1608Metric -> LED_SMD:LED_0805_2012Metric; LCSCPart C2290 -> C2297
- Q1: renamed from Q5; footprint (none) -> Package_TO_SOT_SMD:SOT-23; LCSCPart (none) -> C2143
- R16: renamed from R13; footprint (none) -> Resistor_SMD:R_0603_1608Metric; LCSCPart (none) -> C23182
- R17: renamed from R16; footprint (none) -> Resistor_SMD:R_0603_1608Metric; LCSCPart (none) -> C23182
- R18: renamed from R100; footprint (none) -> Resistor_SMD:R_0603_1608Metric; LCSCPart (none) -> C23182
- R24: renamed from R93; footprint (none) -> Resistor_SMD:R_0603_1608Metric; LCSCPart (none) -> C23182
- R27: renamed from R97; footprint (none) -> Resistor_SMD:R_0603_1608Metric; LCSCPart (none) -> C23182
- R28: renamed from R7; footprint (none) -> Resistor_SMD:R_0603_1608Metric; LCSCPart (none) -> C22962
- R29: renamed from R98; footprint (none) -> Resistor_SMD:R_0603_1608Metric; LCSCPart (none) -> C23182
- R3: renamed from R21; footprint (none) -> Resistor_SMD:R_0603_1608Metric; LCSCPart (none) -> C22962
- R32: renamed from R84; footprint (none) -> Resistor_SMD:R_0603_1608Metric; LCSCPart (none) -> C14676
- R33: renamed from R90; footprint (none) -> Resistor_SMD:R_0603_1608Metric; LCSCPart (none) -> C23182
- R34: renamed from R92; footprint (none) -> Resistor_SMD:R_0603_1608Metric; LCSCPart (none) -> C23182
- R35: renamed from R99; footprint (none) -> Resistor_SMD:R_0603_1608Metric; LCSCPart (none) -> C23182
- R40: renamed from R88; footprint (none) -> Resistor_SMD:R_0603_1608Metric; LCSCPart (none) -> C14676
- R41: renamed from R28; footprint Resistor_SMD:R_2512_6332Metric -> Resistor_SMD:R_0402_1005Metric; LCSCPart C127692 -> C25744
- R42: renamed from R96; footprint Resistor_SMD:R_2512_6332Metric -> Resistor_SMD:R_0603_1608Metric; LCSCPart C127692 -> C23182
- R43: renamed from R25; footprint (none) -> Resistor_SMD:R_0805_2012Metric; LCSCPart (none) -> C17477
- R45: renamed from R29; footprint Resistor_SMD:R_2512_6332Metric -> Resistor_SMD:R_0603_1608Metric; LCSCPart C127692 -> C14676
- R46: renamed from R11; footprint (none) -> Resistor_SMD:R_0402_1005Metric; LCSCPart (none) -> C25744
- R47: renamed from R2; footprint (none) -> Resistor_SMD:R_0603_1608Metric; LCSCPart (none) -> C23182
- R48: renamed from R89; footprint Resistor_SMD:R_2512_6332Metric -> Resistor_SMD:R_0603_1608Metric; LCSCPart C127692 -> C14676
- R49: renamed from R27; footprint Resistor_SMD:R_2512_6332Metric -> Resistor_SMD:R_0402_1005Metric; LCSCPart C127692 -> C25744
- R50: renamed from R15; footprint (none) -> Resistor_SMD:R_0603_1608Metric; LCSCPart (none) -> C23182
- R51: renamed from R26; footprint Resistor_SMD:R_2512_6332Metric -> Resistor_SMD:R_0603_1608Metric; LCSCPart C127692 -> C14676
- renumbered C55 to C1, C57 to C11, C58 to C12, C63 to C13, C59 to C14, C60 to C15, C66 to C16, C67 to C17, C68 to C18, C69 to C19, C74 to C2, C72 to C20, C61 to C21, C64 to C22, C73 to C23, C62 to C24, C65 to C25, C7 to C26, C8 to C27, C2 to C28, C53 to C29, C70 to C3, C3 to C30, C4 to C31, C9 to C32, C5 to C33, C11 to C34, C1 to C4, C75 to C5, C71 to C6, C54 to C7, C6 to C8, C56 to C9, CON to CON1, D3 to D2, D5 to D3, D18 to D5, D19 to D6, D2 to D8, D4 to D9, FB2 to FB1, L2 to L1, L1 to L2, Q6 to Q2, Q7 to Q3, R85 to R1, R19 to R10, R91 to R11, R3 to R12, R20 to R13, R9 to R14, R10 to R15, R80 to R19, R86 to R2, R81 to R22, R18 to R23, R95 to R26, R24 to R30, R82 to R31, R23 to R36, R83 to R37, R8 to R38, R1 to R39, R94 to R4, R12 to R44, R87 to R5, R79 to R6, R5 to R7, R6 to R8, R22 to R9, SW11 to SW2, SW12 to SW3, SW10 to SW4, SW9 to SW5, U17 to U1, U16 to U2, U5 to U4, U1 to U5, U2 to U6, U6 to U7, U4 to U8, Y3 to Y1, Y4 to Y2
Connections:
- net BCK5_EN: now also R25.1
- net BCOUT: now also R21.2
- net LGND: now also R16.2
- net LVCC: now also R17.2
- net SW_BOOT0: now also R20.1; no longer SW2.2 (B)
- new net: R20.2, SW2.2 (B)
- new net: R21.1, R25.2
Other:
- moved on the sheet: C10, D2, D3, R14, R15, R16, R17, SW1

Commit message: application
Parts:
- TH1: footprint (none) -> Resistor_SMD:R_0603_1608Metric; LCSCPart (none) -> C13564
Changed lines of the file:
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@@
 			)
 		)
-		(property "Footprint" ""
+		(property "Footprint" "Resistor_SMD:R_0603_1608Metric"
 			(at 73.66 93.98 0)
 			(effects
@@
 			(at 74.93 93.98 0)
 			(effects
+				(font
+					(size 1.27 1.27)
+				)
+				(hide yes)
+			)
+		)
+		(property "LCSCPart" "C13564"
+			(at 74.93 93.98 0)
+			(effects

Commit message: application
Parts:
- added J1, J2, J3, J4, J5: Conn_01x01_Pin, fpl:EPMM, symbol Connector:Conn_01x01_Pin
- added NT1, NT2, NT3: NetTie_2, NetTie:NetTie-2_SMD_Pad0.5mm, symbol Device:NetTie_2
- BAT1: footprint fpl:BAT-TH_BH-18650-A5BJ003 -> fpl:BATTERY-SMD_18650-1S-L77.1-W20.7-1
- SW1, SW2, SW5: footprint (none) -> fpl:SW-SMD_K3-1235S-K1; LCSCPart (none) -> C92660
- SW3, SW4: footprint (none) -> fpl:SW-TH_5P-L6.0-W6.0-P4.50-LS6.5; LCSCPart (none) -> C470256
Connections:
- net BATSYS: now also J4.1 (Pin_1)
- net BCKOUT33: now also R30.2, R31.1, R36.1, R37.1, J1.1 (Pin_1)
- net BCKOUT5: now also J2.1 (Pin_1)
- net BCOUT: now also U4.11 (OUT)
- net GND: now also J5.1 (Pin_1), NT1.2, NT2.1, NT3.1; no longer C18.2, C19.1, R30.2, R31.1, R36.1, R37.1, Y2.2, Y2.4
- net GNDA: now also NT1.1
- net VBUS: now also J3.1 (Pin_1)
- net USB_D+: now reaches U3.4, U5.8 (D+)
- net USB_D-: now reaches U3.6, U5.7 (D-)
- net +USB_DESP renamed USB_DESP+
- net +USB_DSTM renamed USB_DSTM+
- net -USB_DESP renamed USB_DESP-
- net -USB_DSTM renamed USB_DSTM-
- new net GNDHSC: C18.2, C19.1, NT2.2, Y2.2, Y2.4
- new net GNDLSC: NT3.2
- no-connect marks 19 -> 20
Other:
- note added: "Misc"

Commit message: application
Parts:
- added C37: 10u, Capacitor_SMD:C_0805_2012Metric, symbol Device:C
- C5: value 22u -> 10u; LCSCPart C45783 -> C15850
Connections:
- net BCKOUT33: now also C37.2
- net GND: now also C37.1
Other:
- moved on the sheet: D4, R18
