File: device/hw/$pr/medmentum.kicad_sch (KiCad schematic)
At the start: 131 parts, among them CON1 ZX-IDC2.54-2-13PZZ, J1 Conn_01x01_Pin, J2 Conn_01x01_Pin, J3 Conn_01x01_Pin, J4 Conn_01x01_Pin, J5 Conn_01x01_Pin, Q1 PNP, Q2 NPN, Q3 NPN, SW1 SW_SPDT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

Commit message: application
Parts:
- added H1, H2, H3, H4: ~, MountingHole:MountingHole_2.5mm, symbol Mechanical:MountingHole
- SW3, SW4: footprint fpl:SW-TH_5P-L6.0-W6.0-P4.50-LS6.5 -> fpl:KEY-SMD_4P-L6.0-W6.0-P4.50-LS10.0; LCSCPart C470256 -> C83916
Other:
- note added: "Montažne Tačke"

Commit message: application
Parts:
- removed H4: ~, MountingHole:MountingHole_2.5mm, symbol Mechanical:MountingHole
Changed lines of the file:
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@@
 	(rectangle
 		(start 269.748 66.04)
-		(end 282.194 88.392)
+		(end 282.194 83.82)
 		(stroke
 			(width 0)
@@
 					(unit 1)
 				)
-			)
-		)
-	)
-	(symbol
-		(lib_id "Mechanical:MountingHole")
-		(at 275.59 85.09 0)
-		(unit 1)
-		(exclude_from_sim yes)
-		(in_bom no)
-		(on_board yes)
-		(dnp no)
-		(fields_autoplaced yes)
-		(property "Reference" "H4"
-			(at 278.13 83.8199 0)
-			(effects
-				(font
-					(size 1.27 1.27)
-				)
-				(justify left)
-			)
-		)
-		(property "Value" "~"
-			(at 278.13 86.3599 0)
-			(effects
-				(font
-					(size 1.27 1.27)
-				)
-				(justify left)
-			)
-		)
-		(property "Footprint" "MountingHole:MountingHole_2.5mm"
-			(at 275.59 85.09 0)
-			(effects
-				(font
-					(size 1.27 1.27)
-				)
-				(hide yes)
-			)
-		)
-		(property "Datasheet" "~"
-			(at 275.59 85.09 0)
-			(effects
-				(font
-					(size 1.27 1.27)
-				)
-				(hide yes)
-			)
-		)
-		(property "Description" "Mounting Hole without connection"
-			(at 275.59 85.09 0)
-			(effects
-				(font
-					(size 1.27 1.27)
-				)
-				(hide yes)
-			)
-		)
-		(instances
-			(project "medmentum"
-				(path "/ead52261-b3da-41ef-908f-3daaabe10954"
-					(reference "H4")
-					(unit 1)
-				)

Commit message: application
Connections:
- net CONFSW: now also CON1.14; no longer U7.41 (PB5)
- net CONFSW_DB: now also U7.41 (PB5); no longer CON1.14
- net HOSW: now also CON1.16; no longer U7.45 (PB8)
- net HOSW_DB: now also U7.45 (PB8); no longer CON1.16
Changed lines of the file:
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@@
 	(wire
 		(pts
-			(xy 196.85 100.33) (xy 191.77 100.33)
+			(xy 198.12 100.33) (xy 191.77 100.33)
 		)
 		(stroke
@@
 	(wire
 		(pts
-			(xy 195.58 92.71) (xy 191.77 92.71)
+			(xy 196.85 92.71) (xy 191.77 92.71)
 		)
 		(stroke
@@
 	(polyline
 		(pts
-			(xy 198.12 86.36) (xy 198.12 106.68)
+			(xy 199.39 86.36) (xy 199.39 106.68)
 		)
 		(stroke
@@
 	(polyline
 		(pts
-			(xy 198.12 106.68) (xy 214.63 106.68)
+			(xy 199.39 106.68) (xy 214.63 106.68)
 		)
 		(stroke
@@
 	(polyline
 		(pts
-			(xy 198.12 86.36) (xy 214.63 86.36)
+			(xy 199.39 86.36) (xy 214.63 86.36)
 		)
 		(stroke
@@
 	(wire
 		(pts
-			(xy 264.16 90.17) (xy 257.81 90.17)
+			(xy 261.62 90.17) (xy 257.81 90.17)
 		)
 		(stroke
@@
 	(wire
 		(pts
-			(xy 262.89 92.71) (xy 257.81 92.71)
+			(xy 261.62 92.71) (xy 257.81 92.71)
 		)
 		(stroke
@@
 	(text "TIM4"
 		(exclude_from_sim no)
-		(at 198.374 90.17 0)
+		(at 198.12 90.17 0)
 		(effects
 			(font
@@
 		)
 	)
-	(label "HOSW_DB"
-		(at 262.89 92.71 180)
+	(label "CONFSW"
+		(at 261.62 90.17 180)
 		(effects
 			(font
@@
 		)
 	)
-	(label "HOSW"
-		(at 195.58 92.71 180)
-		(effects
-			(font
-				(size 0.635 0.635)
-				(thickness 0.127)
-				(bold yes)
-			)
-			(justify right bottom)
-		)
-	)
 	(label "USB_DSTM-"
 		(at 95.25 27.94 180)
@@
 		)
 	)
+	(label "HOSW"
+		(at 261.62 92.71 180)
+		(effects
+			(font
+				(size 0.635 0.635)
+				(thickness 0.127)
+				(bold yes)
+			)
+			(justify right bottom)
+		)
+	)
 	(label "BUZPWM"
 		(at 196.85 134.62 180)
@@
 		)
 	)
+	(label "HOSW_DB"
+		(at 196.85 92.71 180)
+		(effects
+			(font
+				(size 0.635 0.635)
+				(thickness 0.127)
+				(bold yes)
+			)
+			(justify right bottom)
+		)
+	)
 	(label "+USB_D"
 		(at 33.02 33.02 0)
@@
 		)
 	)
-	(label "CONFSW_DB"
-		(at 264.16 90.17 180)
-		(effects
-			(font
-				(size 0.635 0.635)
-				(thickness 0.127)
-				(bold yes)
-			)
-			(justify right bottom)
-		)
-	)
 	(label "SERVOPWM6"
 		(at 198.12 152.4 180)
@@
 		)
 	)
+	(label "CONFSW_DB"
+		(at 198.12 100.33 180)
+		(effects
+			(font
+				(size 0.635 0.635)
+				(thickness 0.127)
+				(bold yes)
+			)
+			(justify right bottom)
+		)
+	)
 	(label "CHG_PGOOD"
 		(at 97.79 90.17 180)
@@
 		(effects
 			(font
-				(size 0.635 0.635)
-				(thickness 0.127)
-				(bold yes)
-			)
-			(justify right bottom)
-		)
-	)
-	(label "CONFSW"
-		(at 196.85 100.33 180)
-		(effects
-			(font

Commit message: application
Parts:
- removed NT2, NT3: NetTie_2, NetTie:NetTie-2_SMD_Pad0.5mm, symbol Device:NetTie_2
- C22: value 4.7u -> 1u; footprint Capacitor_SMD:C_0805_2012Metric -> Capacitor_SMD:C_0603_1608Metric; LCSCPart C1779 -> C15849
Connections:
- net +USB_D is gone; now on net USB_D+: U3.3, USB1.10 (D+), USB1.8 (D+)
- net -USB_D is gone; now on net USB_D-: U3.1, USB1.7 (D-), USB1.9 (D-)
- net GNDHSC is gone; now on net GND: C18.2, C19.1, Y2.2, Y2.4
- net GND: no longer R28.1, R3.1
- net LGND: now also R28.1, R3.1
- no-connect marks 20 -> 21

Commit message: application
Connections:
- net SW_BOOT0: no longer D8.1 (K), D9.2 (A), R46.1, SW5.2 (B)
- net USB_SLC: now also R14.2; no longer R15.2
- net at D2.2 (A), D3.1 (K), SW1.2 (B): now also R15.1; no longer R14.1
- net at R46.2: now also U8.23 (IO9); no longer R43.1
- net at R43.2: now also R46.1; no longer U8.23 (IO9)
- new net: R14.1, R15.2
- new net SW_BOOTE0: D8.1 (K), D9.2 (A), R43.1, SW5.2 (B)

Commit message: application
Parts:
- BAT1: LCSCPart C5371778 -> C2988620
Connections:
- net USB_D+: no longer U3.4, U5.8 (D+)
- net USB_D-: no longer U3.6, U5.7 (D-)
- new net USB_DOUT+: U3.4, U5.8 (D+)
- new net USB_DOUT-: U3.6, U5.7 (D-)
Changed lines of the file:
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@@
 		)
 	)
-	(label "USB_D-"
+	(label "USB_DOUT-"
 		(at 67.31 30.48 0)
 		(effects
@@
 		)
 	)
-	(label "USB_D+"
+	(label "USB_DOUT+"
 		(at 67.31 33.02 0)
 		(effects
@@
 			)
 		)
-		(property "LCSCPart" "C5371778"
+		(property "LCSCPart" "C2988620"
 			(at 85.09 143.51 0)
 			(effects
