File: device/hw/$pr/medmentum.kicad_pcb (KiCad board)
At the start: 2 copper layers, 2 parts, among them U1 BQ27441DRZR-G1B, U2 BQ24074RGTR

Commit message: *
Parts:
- added BAT1: Battery_Cell, Battery:BatteryHolder_MPD_BH-18650-PC2, B.Cu at (147.0, 133.0)
- added FB1: 100R@100MHz, Inductor_SMD:L_0805_2012Metric, F.Cu at (142.0, 119.8)
- added U3: TPS62082DSGR, fpl:TPS62082DSGR, F.Cu at (151.5, 105.8)
- added U4: BQ27441DRZR-G1B, fpl:BQ27441DRZR-G1B, F.Cu at (144.5, 98.7)
- added U5: STM32F411CEU6, fpl:STM32F411CEU6, F.Cu at (144.9, 113.8)
- added USB1: USB-310F-B-SU, fpl:USB-310F-B-SU, F.Cu at (147.0, 139.3)
- U1: value BQ27441DRZR-G1B -> TPS63002DRCT; footprint fpl:BQ27441DRZR-G1B -> fpl:TPS63002DRCR
- U2: value BQ24074RGTR -> BQ24074RGTR
- moved U2 24.5 mm to (143.2, 104.9)
- moved U1 21.3 mm to (150.6, 98.9)
Connections:
- net /South Bridge/Battery Managment System/VBSIN renamed VBUS
- net Net-(U2-BAT-Pad2) renamed BATSYS
- U1 pad 1: unconnected-(U1-SDA-Pad1) -> BCKOUT5
- U1 pad 10: unconnected-(U1-BIN-Pad10) -> BCKOUT5
- U1 pad 11: (no net) -> GNDD
- U1 pad 12: unconnected-(U1-GPOUT-Pad12) -> (no net)
- U1 pad 13: unconnected-(U1-EXP-Pad13) -> (no net)
- U1 pad 2: unconnected-(U1-SCL-Pad2) -> Net-(U1-L2)
- U1 pad 3: unconnected-(U1-VSS-Pad3) -> GNDD
- U1 pad 4: (no net) -> Net-(U1-L1)
- U1 pad 5: unconnected-(U1-VDD-Pad5) -> BCOUT
- U1 pad 6: unconnected-(U1-BAT-Pad6) -> Net-(U1-EN)
- U1 pad 7: unconnected-(U1-SRN-Pad7) -> Net-(U1-EN)
- U1 pad 8: unconnected-(U1-SRP-Pad8) -> Net-(U1-EN)
- U1 pad 9: (no net) -> GNDD
- U2 pad 1: unconnected-(U2-TS-Pad1) -> /South Bridge/Battery Managment System/TS
- U2 pad 10: /South Bridge/Battery Managment System/BCOUT -> BCOUT
- U2 pad 11: /South Bridge/Battery Managment System/BCOUT -> unconnected-(U2-OUT-Pad11)
- U2 pad 12: unconnected-(U2-ILIM-Pad12) -> /South Bridge/Battery Managment System/ILIM
- U2 pad 14: unconnected-(U2-TMR-Pad14) -> GNDD
- U2 pad 15: unconnected-(U2-ITERM-Pad15) -> /South Bridge/Battery Managment System/ITERM
- U2 pad 16: unconnected-(U2-ISET-Pad16) -> /South Bridge/Battery Managment System/ISET
- U2 pad 4: unconnected-(U2-~{CE}-Pad4) -> /South Bridge/Battery Managment System/CHG_#CE
- U2 pad 5: unconnected-(U2-EN2-Pad5) -> BCOUT
- U2 pad 6: unconnected-(U2-EN1-Pad6) -> GNDD
- U2 pad 7: unconnected-(U2-~{PGOOD}-Pad7) -> /South Bridge/Battery Managment System/CHG_#PGOOD
- U2 pad 9: unconnected-(U2-~{CHG}-Pad9) -> /South Bridge/Battery Managment System/CHG_#CHG
Other:
- board outline added: 21 x 86 mm

Commit message: application
Parts:
- added U6: USBLC6-2SC6, fpl:USBLC6-2SC6, F.Cu at (187.7, 87.0)
- added U7: TS3USB221ARSER, fpl:TS3USB221ARSER, F.Cu at (186.2, 90.7)
- added U8: ESP32-C3-MINI-1-H4, fpl:ESP32-C3-MINI-1-H4, F.Cu at (146.2, 82.9)
- added Y1: 18pF, Crystal:Crystal_SMD_3225-4Pin_3.2x2.5mm, F.Cu at (187.1, 77.2)
- added Y2: 12.5pF, Crystal:Crystal_SMD_3215-2Pin_3.2x1.5mm, F.Cu at (187.0, 81.1)
Connections:
- net Net-(U5-VREF+) renamed /South Bridge/STM32 MCU/VDDA
- net VBUS renamed /South Bridge/Battery Managment System/VBSIN
- U1 pad 1: BCKOUT5 -> /South Bridge/Battery Managment System/BCK5_VOUT
- U1 pad 10: BCKOUT5 -> /South Bridge/Battery Managment System/BCK5_VOUT
- U5 pad 10: unconnected-(U5-PA0-WKUP-Pad10) -> /South Bridge/STM32 MCU/PWM5
- U5 pad 16: unconnected-(U5-PA6-Pad16) -> /South Bridge/STM32 MCU/PWM1
- U5 pad 17: unconnected-(U5-PA7-Pad17) -> /South Bridge/STM32 MCU/PWM2
- U5 pad 18: unconnected-(U5-PB0-Pad18) -> /South Bridge/STM32 MCU/PWM3
- U5 pad 19: unconnected-(U5-PB1-Pad19) -> /South Bridge/STM32 MCU/PWM4
- U5 pad 21: unconnected-(U5-PB10-Pad21) -> /South Bridge/STM32 MCU/IICGAUG_SCL
- U5 pad 3: unconnected-(U5-PC14-OSC32_IN-Pad3) -> /South Bridge/STM32 MCU/LSE_IN
- U5 pad 30: unconnected-(U5-PA9-Pad30) -> /South Bridge/STM32 MCU/UARTTX_ESP
- U5 pad 31: unconnected-(U5-PA10-Pad31) -> /South Bridge/STM32 MCU/UARTRX_ESP
- U5 pad 32: unconnected-(U5-PA11-Pad32) -> /South Bridge/STM32 MCU/-USB_DSTM
- U5 pad 33: unconnected-(U5-PA12-Pad33) -> /South Bridge/STM32 MCU/+USB_DSTM
- U5 pad 39: unconnected-(U5-PB3-Pad39) -> /South Bridge/STM32 MCU/IICGAUG_SDA
- U5 pad 4: unconnected-(U5-PC15-OSC32_OUT-Pad4) -> /South Bridge/STM32 MCU/LSE_OUT
- U5 pad 42: unconnected-(U5-PB6-Pad42) -> /South Bridge/STM32 MCU/IICDISP_SCL
- U5 pad 43: unconnected-(U5-PB7-Pad43) -> /South Bridge/STM32 MCU/IICDISP_SDA
- U5 pad 44: unconnected-(U5-BOOT0-Pad44) -> /South Bridge/STM32 MCU/BOOT0
- U5 pad 5: Net-(U5-PH0-OSC_IN) -> /South Bridge/STM32 MCU/HSE_IN
- U5 pad 6: Net-(U5-PH1-OSC_OUT) -> /South Bridge/STM32 MCU/HSE_OUT
- U5 pad 7: unconnected-(U5-NRST-Pad7) -> /South Bridge/STM32 MCU/NRST

Commit message: application
Parts:
- removed BAT1: Battery_Cell, Battery:BatteryHolder_MPD_BH-18650-PC2
- removed FB1: 100R@100MHz, Inductor_SMD:L_0805_2012Metric
- removed U1: TPS63002DRCT, fpl:TPS63002DRCR
- removed U2: BQ24074RGTR, fpl:BQ24074RGTR
- removed U3: TPS62082DSGR, fpl:TPS62082DSGR
- removed U4: BQ27441DRZR-G1B, fpl:BQ27441DRZR-G1B
- removed U5: STM32F411CEU6, fpl:STM32F411CEU6
- removed U6: USBLC6-2SC6, fpl:USBLC6-2SC6
- removed U7: TS3USB221ARSER, fpl:TS3USB221ARSER
- removed U8: ESP32-C3-MINI-1-H4, fpl:ESP32-C3-MINI-1-H4
- removed USB1: USB-310F-B-SU, fpl:USB-310F-B-SU
- removed Y1: 18pF, Crystal:Crystal_SMD_3225-4Pin_3.2x2.5mm
- removed Y2: 12.5pF, Crystal:Crystal_SMD_3215-2Pin_3.2x1.5mm
- added G***: LOGO, LOGO, F.Cu at (179.0, 95.0)
- added G***: LOGO, LOGO, F.Cu at (89.5, 93.5)
Other:
- board size 21 x 86 mm -> 40 x 100 mm

Commit message: application
Parts:
- removed the G*** at (179.0, 95.0)
- added BAT1: 2000mAh, fpl:BAT-TH_BH-18650-A5BJ003, F.Cu at (222.0, 101.7)
- added C1: 100n, Capacitor_SMD:C_0603_1608Metric, F.Cu at (165.1, 27.7)
- added C10: 1u, Capacitor_SMD:C_0603_1608Metric, F.Cu at (37.9, 43.3)
- added C11: 1u, Capacitor_SMD:C_0603_1608Metric, F.Cu at (41.9, 35.7)
- added C12: 4.7u, Capacitor_SMD:C_0805_2012Metric, F.Cu at (81.5, 65.3)
- added C13: 100n, Capacitor_SMD:C_0603_1608Metric, F.Cu at (77.3, 55.8)
- added C14: 100n, Capacitor_SMD:C_0603_1608Metric, F.Cu at (77.3, 58.3)
- added C15: 100n, Capacitor_SMD:C_0603_1608Metric, F.Cu at (77.3, 60.8)
- added C16: 100n, Capacitor_SMD:C_0603_1608Metric, F.Cu at (77.3, 63.3)
- added C17: 100n, Capacitor_SMD:C_0603_1608Metric, F.Cu at (77.3, 65.8)
- added C18: 100n, Capacitor_SMD:C_0603_1608Metric, F.Cu at (77.3, 68.3)
- added C19: 4.7u, Capacitor_SMD:C_0805_2012Metric, F.Cu at (81.5, 68.3)
- added C2: 4.7u, Capacitor_SMD:C_0805_2012Metric, F.Cu at (33.6, 36.0)
- added C20: 4.7u, Capacitor_SMD:C_0805_2012Metric, F.Cu at (81.5, 71.3)
- added C21: 100n, Capacitor_SMD:C_0603_1608Metric, F.Cu at (77.3, 70.8)
- added C22: 5p, Capacitor_SMD:C_0402_1005Metric, F.Cu at (85.1, 64.8)
- added C23: 5p, Capacitor_SMD:C_0402_1005Metric, F.Cu at (85.1, 66.8)
- added C24: 16p, Capacitor_SMD:C_0402_1005Metric, F.Cu at (85.1, 68.7)
- added C25: 16p, Capacitor_SMD:C_0402_1005Metric, F.Cu at (85.1, 70.7)
- added C26: 100n, Capacitor_SMD:C_0603_1608Metric, F.Cu at (77.3, 73.4)
- added C27: 4.7u, Capacitor_SMD:C_0805_2012Metric, F.Cu at (81.5, 74.3)
- added C28: 4.7u, Capacitor_SMD:C_0805_2012Metric, F.Cu at (140.7, 81.1)
- added C29: 100n, Capacitor_SMD:C_0603_1608Metric, F.Cu at (155.4, 63.0)
- added C3: 1u, Capacitor_SMD:C_0603_1608Metric, F.Cu at (37.9, 38.2)
- added C30: 100n, Capacitor_SMD:C_0603_1608Metric, F.Cu at (155.4, 65.5)
- added C31: 100n, Capacitor_SMD:C_0603_1608Metric, F.Cu at (155.4, 68.0)
- added C32: 100n, Capacitor_SMD:C_0603_1608Metric, F.Cu at (155.4, 70.6)
- added C33: 1u, Capacitor_SMD:C_0603_1608Metric, F.Cu at (155.4, 73.1)
- added C4: 10u, Capacitor_SMD:C_0805_2012Metric, F.Cu at (33.6, 39.0)
- added C5: 10u, Capacitor_SMD:C_0805_2012Metric, F.Cu at (33.6, 42.0)
- added C6: 10u, Capacitor_SMD:C_0805_2012Metric, F.Cu at (33.6, 45.0)
- added C7: 100n, Capacitor_SMD:C_0603_1608Metric, F.Cu at (37.9, 40.8)
- added C8: 10u, Capacitor_SMD:C_0805_2012Metric, F.Cu at (33.6, 48.0)
- added C9: 22u, Capacitor_SMD:C_0805_2012Metric, F.Cu at (33.6, 51.0)
- added CON1: ZX-IDC2.54-2-13PZZ, fpl:IDC-TH_26P-P2.54_ZX-IDC2.54-2-13PZZ, F.Cu at (236.3, 78.3)
- added D2: LED, LED_SMD:LED_0603_1608Metric, F.Cu at (72.9, 42.3)
- added FB1: 100R@100MHz, Inductor_SMD:L_0805_2012Metric, F.Cu at (91.4, 59.3)
- added L1: 2.2u, Inductor_SMD:L_1008_2520Metric, F.Cu at (67.6, 49.9)
- added L2: 1u, Capacitor_SMD:C_0603_1608Metric, F.Cu at (41.9, 38.2)
- added Q1: NPN, Package_TO_SOT_SMD:SOT-23, F.Cu at (42.5, 67.0)
- added R10: 5.1k 1%, Resistor_SMD:R_0402_1005Metric, F.Cu at (185.0, 31.4)
- added R11: 2.7K, Resistor_SMD:R_0603_1608Metric, F.Cu at (45.9, 35.7)
- added R12: 5.1k 1%, Resistor_SMD:R_0402_1005Metric, F.Cu at (187.9, 27.4)
- added R13: 820, Resistor_SMD:R_0603_1608Metric, F.Cu at (45.9, 38.2)
- added R14: 100k, Resistor_SMD:R_0603_1608Metric, F.Cu at (45.9, 40.8)
- added R15: 100k, Resistor_SMD:R_0603_1608Metric, F.Cu at (45.9, 43.3)
- added R17: 10k, Resistor_SMD:R_0402_1005Metric, F.Cu at (187.9, 29.4)
- added R18: 0, Resistor_SMD:R_0805_2012Metric, F.Cu at (200.3, 31.5)
- added R19: 5.1k, Resistor_SMD:R_0402_1005Metric, F.Cu at (60.7, 39.5)
- added R2: 0, Resistor_SMD:R_0805_2012Metric, F.Cu at (88.8, 65.3)
- added R20: 5.1k, Resistor_SMD:R_0402_1005Metric, F.Cu at (63.6, 35.5)
- added R21: 5.1k, Resistor_SMD:R_0402_1005Metric, F.Cu at (63.6, 37.5)
- added R22: 10m 1% 1W, Resistor_SMD:R_1206_3216Metric, F.Cu at (67.9, 41.4)
- added R24: 10k, Resistor_SMD:R_0402_1005Metric, F.Cu at (63.6, 39.5)
- added R25: 0, Resistor_SMD:R_0805_2012Metric, F.Cu at (88.8, 68.2)
- added R27: 10k, Resistor_SMD:R_0402_1005Metric, F.Cu at (90.6, 61.6)
- added R28: 100k, Resistor_SMD:R_0603_1608Metric, F.Cu at (77.3, 75.9)
- added R29: 10k, Resistor_SMD:R_0402_1005Metric, F.Cu at (154.9, 75.3)
- added R30: 10k, Resistor_SMD:R_0402_1005Metric, F.Cu at (154.9, 77.3)
- added R32: 10k, Resistor_SMD:R_0402_1005Metric, F.Cu at (154.9, 79.3)
- added R33: 1k, Resistor_SMD:R_2512_6332Metric, F.Cu at (35.7, 67.0)
- added R34: 1k, Resistor_SMD:R_2512_6332Metric, F.Cu at (35.7, 71.9)
- added R4: 1.2K, Resistor_SMD:R_0603_1608Metric, F.Cu at (41.9, 40.8)
- added R5: 0, Resistor_SMD:R_0805_2012Metric, F.Cu at (145.1, 81.1)
- added R7: 10k, Resistor_SMD:R_0402_1005Metric, F.Cu at (57.8, 35.5)
- added R8: 10k, Resistor_SMD:R_0402_1005Metric, F.Cu at (185.0, 29.4)
- added R9: 100, Resistor_SMD:R_0603_1608Metric, F.Cu at (41.9, 43.3)
- added U1: TS3USB221ARSER, fpl:TS3USB221ARSER, F.Cu at (199.8, 37.0)
- added U2: BQ24074RGTR, fpl:BQ24074RGTR, F.Cu at (68.3, 37.1)
- added U3: TPS63002DRCT, fpl:TPS63002DRCR, F.Cu at (68.2, 45.5)
- added U4: USBLC6-2SC6, fpl:USBLC6-2SC6, F.Cu at (186.8, 39.0)
- added U5: TPS62082DSGR, fpl:TPS62082DSGR, F.Cu at (73.5, 36.2)
- added U6: BQ27441DRZR-G1B, fpl:BQ27441DRZR-G1B, F.Cu at (60.0, 42.6)
- added U7: STM32F411CEU6, fpl:STM32F411CEU6, F.Cu at (84.5, 59.2)
- added U8: ESP32-C3-MINI-1-H4, fpl:ESP32-C3-MINI-1-H4, F.Cu at (204.0, 68.9)
- added USB1: USB-310F-B-SU, fpl:USB-310F-B-SU, F.Cu at (180.0, 108.0)
- added Y1: 12.5pF, Crystal:Crystal_SMD_3215-2Pin_3.2x1.5mm, F.Cu at (91.6, 56.2)
- added Y2: 18pF, Crystal:Crystal_SMD_3225-4Pin_3.2x2.5mm, F.Cu at (89.2, 71.9)
Other:
- board size 40 x 100 mm -> 14 x 70 mm

Commit message: application
Parts:
- removed G***: LOGO, LOGO
- added BZ1: Buzzer, fpl:BUZ-TH_BD17.0-P10.00-D0.8, F.Cu at (214.6, 151.0)
- added C34: 1u, Capacitor_SMD:C_0603_1608Metric, F.Cu at (86.9, 65.1)
- added C35: 100n, Capacitor_SMD:C_0603_1608Metric, F.Cu at (105.2, 149.1)
- added C36: 100n, Capacitor_SMD:C_0603_1608Metric, F.Cu at (109.2, 126.5)
- added D1: LED, LED_SMD:LED_0805_2012Metric, F.Cu at (261.5, 45.1)
- added D3: LED, LED_SMD:LED_0603_1608Metric, F.Cu at (259.3, 76.8)
- added D4: LED, LED_SMD:LED_0805_2012Metric, F.Cu at (73.4, 116.1)
- added D5: LED, LED_SMD:LED_0603_1608Metric, F.Cu at (167.1, 103.9)
- added D6: LED, LED_SMD:LED_0603_1608Metric, F.Cu at (167.1, 106.5)
- added D7: LED, LED_SMD:LED_0805_2012Metric, F.Cu at (261.5, 51.2)
- added D8: LED, LED_SMD:LED_0603_1608Metric, F.Cu at (149.2, 66.1)
- added D9: LED, LED_SMD:LED_0603_1608Metric, F.Cu at (149.2, 68.7)
- added J1: Conn_01x01_Pin, fpl:EPMM, F.Cu at (261.8, 30.1)
- added J2: Conn_01x01_Pin, fpl:EPMM, F.Cu at (261.8, 33.1)
- added J3: Conn_01x01_Pin, fpl:EPMM, F.Cu at (261.8, 36.1)
- added J4: Conn_01x01_Pin, fpl:EPMM, F.Cu at (261.8, 39.1)
- added J5: Conn_01x01_Pin, fpl:EPMM, F.Cu at (261.8, 42.1)
- added NT1: NetTie_2, NetTie:NetTie-2_SMD_Pad0.5mm, F.Cu at (116.3, 151.1)
- added NT2: NetTie_2, NetTie:NetTie-2_SMD_Pad0.5mm, F.Cu at (246.5, 20.5)
- added NT3: NetTie_2, NetTie:NetTie-2_SMD_Pad0.5mm, F.Cu at (246.5, 22.0)
- added Q2: NPN, Package_TO_SOT_SMD:SOT-23, F.Cu at (108.8, 115.3)
- added Q3: NPN, Package_TO_SOT_SMD:SOT-23, F.Cu at (209.0, 137.9)
- added R1: 5.1k, Resistor_SMD:R_0402_1005Metric, F.Cu at (114.7, 92.7)
- added R16: 47, Resistor_SMD:R_0603_1608Metric, F.Cu at (220.7, 80.6)
- added R23: 0, Resistor_SMD:R_0805_2012Metric, F.Cu at (80.5, 96.2)
- added R26: 10k, Resistor_SMD:R_0402_1005Metric, F.Cu at (99.6, 95.6)
- added R3: 220, Resistor_SMD:R_0603_1608Metric, F.Cu at (256.7, 45.0)
- added R31: 5.1k, Resistor_SMD:R_0402_1005Metric, F.Cu at (102.5, 93.8)
- added R35: 47, Resistor_SMD:R_0603_1608Metric, F.Cu at (97.3, 108.2)
- added R36: 5.1k, Resistor_SMD:R_0402_1005Metric, F.Cu at (102.7, 107.7)
- added R37: 5.1k, Resistor_SMD:R_0402_1005Metric, F.Cu at (104.6, 93.8)
- added R38: 10k, Resistor_SMD:R_0402_1005Metric, F.Cu at (87.4, 63.3)
- added R39: 10k, Resistor_SMD:R_0402_1005Metric, F.Cu at (87.4, 66.8)
- added R40: 1k, Resistor_SMD:R_0603_1608Metric, F.Cu at (104.6, 114.2)
- added R41: 10k, Resistor_SMD:R_0402_1005Metric, F.Cu at (274.5, 45.5)
- added R42: 47, Resistor_SMD:R_0603_1608Metric, F.Cu at (160.1, 59.0)
- added R43: 0, Resistor_SMD:R_0805_2012Metric, F.Cu at (138.7, 75.3)
- added R44: 10k, Resistor_SMD:R_0402_1005Metric, F.Cu at (99.3, 71.0)
- added R45: 1k, Resistor_SMD:R_0603_1608Metric, F.Cu at (117.2, 134.1)
- added R46: 10k, Resistor_SMD:R_0402_1005Metric, F.Cu at (141.2, 75.7)
- added R47: 47, Resistor_SMD:R_0603_1608Metric, F.Cu at (152.9, 66.1)
- added R48: 1k, Resistor_SMD:R_0603_1608Metric, F.Cu at (204.9, 142.9)
- added R49: 10k, Resistor_SMD:R_0402_1005Metric, F.Cu at (274.5, 51.4)
- added R50: 47, Resistor_SMD:R_0603_1608Metric, F.Cu at (152.9, 68.8)
- added R51: 1k, Resistor_SMD:R_0603_1608Metric, F.Cu at (117.2, 144.1)
- added R6: 820, Resistor_SMD:R_0603_1608Metric, F.Cu at (94.0, 73.5)
- added SW1: SW_SPDT, fpl:SW-SMD_K3-1235S-K1, F.Cu at (205.5, 68.9)
- added SW2: SW_SPDT, fpl:SW-SMD_K3-1235S-K1, F.Cu at (144.1, 122.8)
- added SW3: SW_Push, fpl:SW-TH_5P-L6.0-W6.0-P4.50-LS6.5, F.Cu at (182.2, 102.5)
- added SW4: SW_Push, fpl:SW-TH_5P-L6.0-W6.0-P4.50-LS6.5, F.Cu at (132.2, 32.8)
- added SW5: SW_SPDT, fpl:SW-SMD_K3-1235S-K1, F.Cu at (107.0, 30.0)
- added TH1: 10K, Resistor_SMD:R_0603_1608Metric, F.Cu at (113.4, 109.2)
- BAT1: footprint fpl:BAT-TH_BH-18650-A5BJ003 -> fpl:BATTERY-SMD_18650-1S-L77.1-W20.7-1; moved to B.Cu
- C1, C32: value 100n -> 1u
- C10, C11, C33: value 1u -> 100n
- C12, C20: value 4.7u -> 100n; footprint Capacitor_SMD:C_0805_2012Metric -> Capacitor_SMD:C_0603_1608Metric
- C13, C7: value 100n -> 4.7u; footprint Capacitor_SMD:C_0603_1608Metric -> Capacitor_SMD:C_0805_2012Metric
- C16, C17: value 100n -> 5p; footprint Capacitor_SMD:C_0603_1608Metric -> Capacitor_SMD:C_0402_1005Metric
- C18: value 100n -> 16p; footprint Capacitor_SMD:C_0603_1608Metric -> Capacitor_SMD:C_0402_1005Metric
- C19: value 4.7u -> 16p; footprint Capacitor_SMD:C_0805_2012Metric -> Capacitor_SMD:C_0402_1005Metric
- C2, C27: value 4.7u -> 10u
- C22, C23: value 5p -> 4.7u; footprint Capacitor_SMD:C_0402_1005Metric -> Capacitor_SMD:C_0805_2012Metric
- C24, C25: value 16p -> 100n; footprint Capacitor_SMD:C_0402_1005Metric -> Capacitor_SMD:C_0603_1608Metric
- C26: value 100n -> 10u; footprint Capacitor_SMD:C_0603_1608Metric -> Capacitor_SMD:C_0805_2012Metric
- C4: value 10u -> 100n; footprint Capacitor_SMD:C_0805_2012Metric -> Capacitor_SMD:C_0603_1608Metric
- C5: value 10u -> 22u
- C6: value 10u -> 1u; footprint Capacitor_SMD:C_0805_2012Metric -> Capacitor_SMD:C_0603_1608Metric
- C9: value 22u -> 4.7u
- L1: value 2.2u -> 1u; footprint Inductor_SMD:L_1008_2520Metric -> Capacitor_SMD:C_0603_1608Metric
- L2: value 1u -> 2.2u; footprint Capacitor_SMD:C_0603_1608Metric -> Inductor_SMD:L_1008_2520Metric
- Q1: value NPN -> PNP
- R10: value 5.1k 1% -> 1.2K; footprint Resistor_SMD:R_0402_1005Metric -> Resistor_SMD:R_0603_1608Metric
- R11: value 2.7K -> 10m 1% 1W; footprint Resistor_SMD:R_0603_1608Metric -> Resistor_SMD:R_1206_3216Metric
- R12: value 5.1k 1% -> 10k
- R13: value 820 -> 10k; footprint Resistor_SMD:R_0603_1608Metric -> Resistor_SMD:R_0402_1005Metric
- R14: value 100k -> 10k; footprint Resistor_SMD:R_0603_1608Metric -> Resistor_SMD:R_0402_1005Metric
- R15: value 100k -> 0; footprint Resistor_SMD:R_0603_1608Metric -> Resistor_SMD:R_0805_2012Metric
- R17, R24, R27, R29: value 10k -> 47; footprint Resistor_SMD:R_0402_1005Metric -> Resistor_SMD:R_0603_1608Metric
- R18, R25: value 0 -> 47; footprint Resistor_SMD:R_0805_2012Metric -> Resistor_SMD:R_0603_1608Metric
- R19: value 5.1k -> 100k; footprint Resistor_SMD:R_0402_1005Metric -> Resistor_SMD:R_0603_1608Metric
- R2, R5: value 0 -> 5.1k; footprint Resistor_SMD:R_0805_2012Metric -> Resistor_SMD:R_0402_1005Metric
- R20: value 5.1k -> 0; footprint Resistor_SMD:R_0402_1005Metric -> Resistor_SMD:R_0805_2012Metric
- R21: value 5.1k -> 47; footprint Resistor_SMD:R_0402_1005Metric -> Resistor_SMD:R_0603_1608Metric
- R22: value 10m 1% 1W -> 100k; footprint Resistor_SMD:R_1206_3216Metric -> Resistor_SMD:R_0603_1608Metric
- R28: value 100k -> 220
- R30: value 10k -> 5.1k
- R32: value 10k -> 1k; footprint Resistor_SMD:R_0402_1005Metric -> Resistor_SMD:R_0603_1608Metric
- R33, R34: value 1k -> 47; footprint Resistor_SMD:R_2512_6332Metric -> Resistor_SMD:R_0603_1608Metric
- R4: value 1.2K -> 10k; footprint Resistor_SMD:R_0603_1608Metric -> Resistor_SMD:R_0402_1005Metric
- R7, R8: value 10k -> 5.1k 1%
- R9: value 100 -> 2.7K
- U1: value TS3USB221ARSER -> TPS62082DSGR; footprint fpl:TS3USB221ARSER -> fpl:TPS62082DSGR
- U2: value BQ24074RGTR -> BQ27441DRZR-G1B; footprint fpl:BQ24074RGTR -> fpl:BQ27441DRZR-G1B
- U3: value TPS63002DRCT -> USBLC6-2SC6; footprint fpl:TPS63002DRCR -> fpl:USBLC6-2SC6
- U4: value USBLC6-2SC6 -> BQ24074RGTR; footprint fpl:USBLC6-2SC6 -> fpl:BQ24074RGTR
- U5: value TPS62082DSGR -> TS3USB221ARSER; footprint fpl:TPS62082DSGR -> fpl:TS3USB221ARSER
- U6: value BQ27441DRZR-G1B -> TPS63002DRCT; footprint fpl:BQ27441DRZR-G1B -> fpl:TPS63002DRCR
- moved R14 230.9 mm to (270.6, 93.7)
- moved R15 229.6 mm to (273.4, 74.4)
- moved C8 229.2 mm to (261.1, 20.5)
- moved C26 196.5 mm to (265.6, 17.5)
- moved C27 191.8 mm to (265.6, 20.5)
- moved D2 189.0 mm to (259.3, 74.2)
- moved BAT1 167.8 mm to (54.2, 102.2), turned to 0 degrees
- moved R20 158.8 mm to (196.1, 123.1)
- moved R18 147.9 mm to (78.7, 115.6)
- moved L2 137.0 mm to (112.5, 155.6)
- moved U1 135.4 mm to (90.1, 116.4), turned to 90 degrees
- moved R24 118.4 mm to (163.1, 103.5)
- moved U6 118.1 mm to (102.3, 152.9)
- moved C10 112.8 mm to (101.2, 136.6)
- moved U8 108.5 mm to (95.6, 64.7)
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Connections:
- BAT1 pad 1: /South Bridge/Battery Managment System/BAT -> /BAT
- C1 pad 1: GNDD -> VBUS
- C1 pad 2: BCKOUT33 -> GNDD
- C10 pad 1: Net-(U6-VDD) -> GNDD
- C10 pad 2: GNDD -> /BCK5_EN
- C11 pad 2: /South Bridge/Battery Managment System/BAT -> VDD
- C13 pad 1: GNDD -> GNDA
- C13 pad 2: VDD -> BCKOUT33
- C16 pad 1: GNDD -> /LSE_IN
- C16 pad 2: VDD -> GNDD
- C17 pad 2: VDD -> /LSE_OUT
- C18 pad 1: GNDD -> /HSE_IN
- C18 pad 2: VDD -> GNDHSC
- C19 pad 1: GNDA -> GNDHSC
- C19 pad 2: BCKOUT33 -> /HSE_OUT
- C2 pad 2: BCOUT -> BCKOUT5
- C20 pad 1: GNDA -> GNDD
- C20 pad 2: /South Bridge/STM32 MCU/VDDASTM -> /NRST
- C21 pad 1: GNDA -> GNDD
- C21 pad 2: /South Bridge/STM32 MCU/VDDASTM -> VDD
- C22 pad 1: /South Bridge/STM32 MCU/LSE_IN -> GNDA
- C22 pad 2: GNDD -> /VDDASTM
- C23 pad 2: /South Bridge/STM32 MCU/LSE_OUT -> Net-(U7-VCAP_1)
- C24 pad 1: /South Bridge/STM32 MCU/HSE_IN -> GNDD
- C24 pad 2: GNDD -> VDD
- C25 pad 1: GNDD -> GNDA
- C25 pad 2: /South Bridge/STM32 MCU/HSE_OUT -> /VDDASTM
- C26 pad 2: /South Bridge/STM32 MCU/NRST -> BCKOUT5
- C27 pad 2: Net-(U7-VCAP_1) -> BCKOUT5
- C28 pad 1: GNDD -> BCKOUT33
- C28 pad 2: BCKOUT33 -> GNDD
- C29 pad 1: GNDD -> /ENRST
- C29 pad 2: BCKOUT33 -> GNDD
- C3 pad 1: VBUS -> Net-(U2-VDD)
- C30 pad 1: GNDD -> BCKOUT33
- C30 pad 2: BCKOUT33 -> GNDD
- C31 pad 1: GNDD -> BCKOUT33
- C31 pad 2: BCKOUT33 -> GNDD
- C32 pad 1: /North Bridge/ESP32 MCU/ENESP -> /ENRST
- C33 pad 1: GNDD -> BCKOUT33
- C33 pad 2: /North Bridge/ESP32 MCU/ENESP -> GNDD
- C4 pad 2: BCOUT -> BCKOUT33
- C5 pad 2: BCKOUT5 -> BCKOUT33
- C6 pad 2: BCKOUT5 -> /BAT
- C7 pad 2: /South Bridge/Battery Managment System/BCK5_EN -> BCOUT
- C8 pad 2: BCKOUT5 -> BCOUT
- C9 pad 2: BCKOUT33 -> VDD
- CON1 pad 1: /Peripherals/SERVOPWM1 -> /SERVOPWM1
- CON1 pad 10: /Peripherals/SERVOPWM5 -> /IICDISP_SDA
- CON1 pad 11: /Peripherals/IICDISP_SDA -> /SERVOPWM5
- CON1 pad 13: BCKOUT5 -> GNDD
- CON1 pad 14: GNDD -> /CONFSW_DB
- CON1 pad 16: /Peripherals/PANICPWM2 -> /HOSW_DB
- CON1 pad 17: /Peripherals/PANICGPIO -> GNDD
- CON1 pad 18: /Peripherals/PANICPWM1 -> /LEDCHPWM
- CON1 pad 19: /Peripherals/LEDCHPWM -> BCKOUT33
- CON1 pad 2: BCKOUT5 -> /SERVOPWM2
- CON1 pad 20: BCKOUT33 -> /LEDHOPWM
- CON1 pad 22: /Peripherals/CONFSW -> /SERVOPWM6
- CON1 pad 23: /Peripherals/LEDHOPWM -> BCKOUT5
- CON1 pad 24: BCKOUT33 -> GNDD
- CON1 pad 25: BCKOUT33 -> /PANICPWM
- CON1 pad 26: /Peripherals/HOSW -> /PANICGPIO
- CON1 pad 3: /Peripherals/SERVOPWM2 -> /SERVOPWM3
- CON1 pad 4: BCKOUT5 -> /SERVOPWM4
- CON1 pad 5: /Peripherals/SERVOPWM3 -> BCKOUT5
- CON1 pad 7: /Peripherals/SERVOPWM4 -> BCKOUT5
- CON1 pad 9: /Peripherals/IICDISP_SCL -> /IICDISP_SCL
- D2 pad 1: LGND -> Net-(D2-K)
- D2 pad 2: BCKOUT33 -> Net-(D2-A)
- FB1 pad 2: /South Bridge/STM32 MCU/VDDASTM -> /VDDASTM
- L1 pad 1: Net-(U3-L1) -> Net-(U1-SW)
- L1 pad 2: Net-(U3-L2) -> BCKOUT33
- L2 pad 1: Net-(U5-SW) -> Net-(U6-L1)
- L2 pad 2: BCKOUT33 -> Net-(U6-L2)
- Q1 pad 1: Net-(BZ1--) -> LVCC
- Q1 pad 3: GNDD -> BCKOUT33
- R10 pad 1: /South Bridge/Battery Managment System/CC1 -> GNDD
- R10 pad 2: GNDD -> /ILIM
- R11 pad 1: GNDD -> BATSYS
- R11 pad 2: /South Bridge/Battery Managment System/ITERM -> /BAT
- R12 pad 1: /South Bridge/Battery Managment System/CC2 -> GNDD
- R12 pad 2: GNDD -> Net-(U5-~{OE})
- R13 pad 2: /South Bridge/Battery Managment System/ISET -> Net-(U4-~{CE})
- R14 pad 1: BCKOUT33 -> Net-(D2-A)
- R14 pad 2: /South Bridge/Battery Managment System/CHG_#CHG -> Net-(R14-Pad2)
- R15 pad 1: BCKOUT33 -> Net-(R14-Pad2)
- R15 pad 2: /South Bridge/Battery Managment System/CHG_#PGOOD -> /USB_SLC
- R17 pad 2: Net-(R17-Pad2) -> LVCC
- R18 pad 1: Net-(R17-Pad2) -> LGND
- R18 pad 2: /South Bridge/Battery Managment System/USB_SLC -> Net-(D4-K)
- R19 pad 1: /South Bridge/Battery Managment System/FG_SCL -> BCKOUT33
- R19 pad 2: BCKOUT33 -> /CHG_#CHG
- R2 pad 1: Net-(SW2-B) -> /FG_SDA
- R2 pad 2: /South Bridge/STM32 MCU/SW_BOOT0 -> BCKOUT33
- R20 pad 1: /South Bridge/Battery Managment System/FG_SDA -> /SW_BOOT0
- R20 pad 2: BCKOUT33 -> Net-(SW2-B)
- R21 pad 1: /South Bridge/Battery Managment System/FG_GPOUT -> Net-(R21-Pad1)
- R21 pad 2: BCKOUT33 -> BCOUT
- R22 pad 1: BATSYS -> BCKOUT33
- R22 pad 2: /South Bridge/Battery Managment System/BAT -> /CHG_#PGOOD
- R24 pad 1: /South Bridge/Battery Managment System/FG_BIN -> Net-(D5-A)
- R24 pad 2: GNDD -> LVCC
- R25 pad 1: BCKOUT33 -> /BCK5_EN
- R25 pad 2: VDD -> Net-(R21-Pad1)
- R27 pad 1: /South Bridge/STM32 MCU/SW_BOOT0 -> LGND
- R27 pad 2: /South Bridge/STM32 MCU/BOOT0 -> Net-(D6-K)
- R28 pad 1: BCKOUT33 -> GNDD
- R28 pad 2: /South Bridge/STM32 MCU/NRST -> Net-(D7-K)
- R29 pad 1: /North Bridge/ESP32 MCU/ENESP -> Net-(U7-PA3)
- R29 pad 2: BCKOUT33 -> /LEDHOPWM
- R30 pad 1: BCKOUT33 -> /IICDISP_SDA
- R30 pad 2: Net-(U8-IO2) -> BCKOUT33
- R32 pad 1: Net-(U8-IO8) -> Net-(U7-PA14)
- R32 pad 2: BCKOUT33 -> Net-(Q1-B)
- R33 pad 1: Net-(BZ1--) -> /STM_UARTRX
- R33 pad 2: /Peripherals/BUZVCC -> /UARTRX_ESP
- R34 pad 1: /Peripherals/BUZPWM -> /STM_UARTTX
- R34 pad 2: Net-(Q1-B) -> /UARTTX_ESP
- R4 pad 1: GNDD -> /FG_BIN
- R4 pad 2: /South Bridge/Battery Managment System/ILIM -> GNDD
- R5 pad 1: Net-(U8-IO9) -> /FG_GPOUT
- R5 pad 2: Net-(SW5-B) -> BCKOUT33
- R7 pad 1: GNDD -> /CC1
- R7 pad 2: Net-(U2-~{CE}) -> GNDD
- R8 pad 1: GNDD -> /CC2
- R8 pad 2: Net-(U1-~{OE}) -> GNDD
- R9 pad 1: /South Bridge/Battery Managment System/BCK5_EN -> GNDD
- R9 pad 2: BCOUT -> /ITERM
- U1 pad 1: /South Bridge/Battery Managment System/+USB_DSTM -> BCKOUT5
- U1 pad 2: /South Bridge/Battery Managment System/-USB_DSTM -> GNDD
- U1 pad 3: /South Bridge/Battery Managment System/+USB_DESP -> GNDD
- U1 pad 4: /South Bridge/Battery Managment System/-USB_DESP -> unconnected-(U1-FB-Pad4)
- U1 pad 5: GNDD -> BCKOUT33
- U1 pad 6: Net-(U1-~{OE}) -> unconnected-(U1-PG-Pad6)
- U1 pad 7: Net-(U1-D-) -> Net-(U1-SW)
- U1 pad 8: Net-(U1-D+) -> BCKOUT5
- U1 pad 9: /South Bridge/Battery Managment System/USB_SLC -> GNDD
- U2 pad 1: /South Bridge/Battery Managment System/TS -> /FG_SDA
- U2 pad 10: BCOUT -> /FG_BIN
- U2 pad 11: unconnected-(U2-OUT-Pad11) -> (no net)
- U2 pad 12: /South Bridge/Battery Managment System/ILIM -> /FG_GPOUT
- U2 pad 13: VBUS -> GNDD
- U2 pad 2: BATSYS -> /FG_SCL
- U2 pad 3: BATSYS -> GNDD
- U2 pad 4: Net-(U2-~{CE}) -> (no net)
- U2 pad 5: BCOUT -> Net-(U2-VDD)
- U2 pad 6: GNDD -> /BAT
- U2 pad 7: /South Bridge/Battery Managment System/CHG_#PGOOD -> BATSYS
- U2 pad 8: GNDD -> /BAT
- U2 pad 9: /South Bridge/Battery Managment System/CHG_#CHG -> (no net)
- U3 pad 1: BCKOUT5 -> /-USB_D
- U3 pad 2: Net-(U3-L2) -> GNDD
- U3 pad 3: GNDD -> /+USB_D
- U3 pad 4: Net-(U3-L1) -> /USB_D+
- U3 pad 5: BCOUT -> VBUS
- U3 pad 6: /South Bridge/Battery Managment System/BCK5_EN -> /USB_D-
- U4 pad 1: /South Bridge/Battery Managment System/-USB_D -> /TS
- U4 pad 2: GNDD -> BATSYS
- U4 pad 3: /South Bridge/Battery Managment System/+USB_D -> BATSYS
- U4 pad 4: Net-(U1-D+) -> Net-(U4-~{CE})
- U4 pad 5: VBUS -> BCOUT
- U4 pad 6: Net-(U1-D-) -> GNDD
- U5 pad 1: BCKOUT5 -> /USB_DSTM+
- U5 pad 2: GNDD -> /USB_DSTM-
- U5 pad 3: GNDD -> /USB_DESP+
- U5 pad 4: unconnected-(U5-FB-Pad4) -> /USB_DESP-
- U5 pad 5: BCKOUT33 -> GNDD
- U5 pad 6: unconnected-(U5-PG-Pad6) -> Net-(U5-~{OE})
- U5 pad 7: Net-(U5-SW) -> /USB_D-
- U5 pad 8: BCKOUT5 -> /USB_D+
- U5 pad 9: GNDD -> /USB_SLC
- U6 pad 1: /South Bridge/Battery Managment System/FG_SDA -> BCKOUT5
- U6 pad 10: /South Bridge/Battery Managment System/FG_BIN -> BCKOUT5
- U6 pad 11: (no net) -> GNDD
- U6 pad 12: /South Bridge/Battery Managment System/FG_GPOUT -> (no net)
- U6 pad 13: GNDD -> (no net)
- U6 pad 2: /South Bridge/Battery Managment System/FG_SCL -> Net-(U6-L2)
- U6 pad 4: (no net) -> Net-(U6-L1)
- U6 pad 5: Net-(U6-VDD) -> BCOUT
- U6 pad 6: /South Bridge/Battery Managment System/BAT -> /BCK5_EN
- U6 pad 7: BATSYS -> /BCK5_EN
- U6 pad 8: /South Bridge/Battery Managment System/BAT -> /BCK5_EN
- U6 pad 9: (no net) -> GNDD
- U7 pad 10: /South Bridge/STM32 MCU/SERVOPWM5 -> /SERVOPWM5
- U7 pad 11: /South Bridge/STM32 MCU/PANICPWM1 -> /SERVOPWM6
- U7 pad 16: /South Bridge/STM32 MCU/SERVOPWM1 -> /SERVOPWM1
- U7 pad 17: /South Bridge/STM32 MCU/SERVOPWM2 -> /SERVOPWM2
- U7 pad 18: /South Bridge/STM32 MCU/SERVOPWM3 -> /SERVOPWM3
- U7 pad 19: /South Bridge/STM32 MCU/SERVOPWM4 -> /SERVOPWM4
- U7 pad 21: /South Bridge/STM32 MCU/IICGAUG_SCL -> /FG_SCL
- U7 pad 25: /South Bridge/STM32 MCU/PANICGPIO -> /PANICGPIO
- U7 pad 26: /South Bridge/STM32 MCU/FG_GPOUT -> /FG_GPOUT
- U7 pad 27: /South Bridge/STM32 MCU/CHG_PGOOD -> /CHG_#PGOOD
- U7 pad 28: /South Bridge/STM32 MCU/CHG_CHG -> /CHG_#CHG
- U7 pad 29: /South Bridge/STM32 MCU/BUZPWM -> /BUZPWM
- U7 pad 3: /South Bridge/STM32 MCU/LSE_IN -> /LSE_IN
- U7 pad 30: /South Bridge/STM32 MCU/UARTTX_ESP -> /STM_UARTTX
- U7 pad 31: /South Bridge/STM32 MCU/UARTRX_ESP -> /STM_UARTRX
- U7 pad 32: /South Bridge/STM32 MCU/-USB_DSTM -> /USB_DSTM-
- U7 pad 33: /South Bridge/STM32 MCU/+USB_DSTM -> /USB_DSTM+
- U7 pad 34: /South Bridge/STM32 MCU/DISPEN -> unconnected-(U7-PA13-Pad34)
- U7 pad 37: /South Bridge/STM32 MCU/LEDEN -> Net-(U7-PA14)
- U7 pad 39: /South Bridge/STM32 MCU/IICGAUG_SDA -> /FG_SDA
- U7 pad 4: /South Bridge/STM32 MCU/LSE_OUT -> /LSE_OUT
- U7 pad 41: /South Bridge/STM32 MCU/CONFSW -> /CONFSW
- U7 pad 42: /South Bridge/STM32 MCU/IICDISP_SCL -> /IICDISP_SCL
- U7 pad 43: /South Bridge/STM32 MCU/IICDISP_SDA -> /IICDISP_SDA
- U7 pad 44: /South Bridge/STM32 MCU/BOOT0 -> /BOOT0
- U7 pad 45: /South Bridge/STM32 MCU/HOSW -> /HOSW
- U7 pad 46: unconnected-(U7-PB9-Pad46) -> /PANICPWM
- U7 pad 5: /South Bridge/STM32 MCU/HSE_IN -> /HSE_IN
- U7 pad 6: /South Bridge/STM32 MCU/HSE_OUT -> /HSE_OUT
- U7 pad 7: /South Bridge/STM32 MCU/NRST -> /NRST
- U7 pad 9: /South Bridge/STM32 MCU/VDDASTM -> /VDDASTM
- U8 pad 26: /North Bridge/ESP32 MCU/-USB_DESP -> /USB_DESP-
- U8 pad 27: /North Bridge/ESP32 MCU/+USB_DESP -> /USB_DESP+
- U8 pad 30: /North Bridge/ESP32 MCU/UARTTX_ESP -> /UARTTX_ESP
- U8 pad 31: /North Bridge/ESP32 MCU/UARTRX_ESP -> /UARTRX_ESP
- U8 pad 8: /North Bridge/ESP32 MCU/ENESP -> /ENRST
- Y1 pad 1: /South Bridge/STM32 MCU/LSE_OUT -> /LSE_OUT
- Y1 pad 2: /South Bridge/STM32 MCU/LSE_IN -> /LSE_IN
- Y2 pad 1: /South Bridge/STM32 MCU/HSE_IN -> /HSE_IN
- Y2 pad 2: GNDD -> GNDHSC
- Y2 pad 3: /South Bridge/STM32 MCU/HSE_OUT -> /HSE_OUT
- Y2 pad 4: GNDD -> GNDHSC
Routing:
- net /HSE_IN: track 0.00 -> 16.1 mm
- net /HSE_OUT: track 0.00 -> 15.6 mm
- net GNDD: track 0.00 -> 8.84 mm, vias 0 -> 9
- net BCKOUT33: track 0.00 -> 7.05 mm
- net /LSE_OUT: track 0.00 -> 6.37 mm
- net /LSE_IN: track 0.00 -> 6.33 mm
- net /BAT: track 0.00 -> 5.23 mm
- net /-USB_D: track 0.00 -> 5.06 mm
- net /+USB_D: track 0.00 -> 4.39 mm
- net BATSYS: track 0.00 -> 3.63 mm
- net /VDDASTM: track 0.00 -> 3.59 mm, vias 0 -> 1
- net /STM_UARTTX: track 0.00 -> 3.16 mm
- net /STM_UARTRX: track 0.00 -> 3.12 mm
- net Net-(U7-PA2): track 0.00 -> 2.59 mm
- net /FG_SCL: track 0.00 -> 2.27 mm, vias 0 -> 1
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Other:
- board outline removed
- copper layers 2 -> 6
- board text added: "Sig G Sig Pow G S"

Commit message: application
Parts:
- added C37: 10u, Capacitor_SMD:C_0805_2012Metric, F.Cu at (97.7, 91.0)
- C5: value 22u -> 10u
- TH1: moved to B.Cu
- moved J1 234.3 mm to (38.2, 100.3)
- moved J2 234.3 mm to (38.2, 103.3)
- moved J3 234.3 mm to (38.2, 106.3)
- moved J4 234.3 mm to (38.2, 109.3)
- moved J5 234.3 mm to (38.2, 112.3)
- moved R41 196.8 mm to (86.8, 104.8)
- moved C26 190.0 mm to (91.3, 93.2)
- moved C27 189.7 mm to (91.3, 95.4)
- moved C8 180.5 mm to (93.2, 86.8), turned to 180 degrees
- moved BZ1 162.8 mm to (51.8, 155.4), turned to 0 degrees
- moved R15 160.7 mm to (113.5, 58.1)
- moved R14 160.7 mm to (113.3, 60.7)
- moved CON1 134.8 mm to (76.8, 86.3)
- moved D7 128.8 mm to (135.6, 78.5)
- moved SW1 120.5 mm to (123.3, 157.0), turned to 90 degrees
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Connections:
- U6 pad 12: (no net) -> GNDD
- U6 pad 13: (no net) -> GNDD
- U6 pad 14: (no net) -> GNDD
- U6 pad 15: (no net) -> GNDD
Routing:
- net BCOUT: track 0.00 -> 17.6 mm, vias 0 -> 3
- net BATSYS: track 3.63 -> 13.6 mm, vias 0 -> 2
- net /BAT: track 5.23 -> 13.5 mm, vias 0 -> 3
- net BCKOUT5: track 2.14 -> 5.83 mm
- net /BCK5_EN: track 0.00 -> 3.38 mm
- net /STM_UARTTX: track 3.16 -> 0.00 mm
- net /STM_UARTRX: track 3.12 -> 0.00 mm
- net GNDD: track 8.84 -> 11.8 mm, vias 9 -> 8
- net /CHG_#CHG: track 0.00 -> 2.55 mm
- net /FG_SCL: track 2.27 -> 4.79 mm
- net Net-(U6-L2): track 0.00 -> 2.34 mm
- net Net-(U6-L1): track 0.00 -> 2.34 mm
- net /CHG_#PGOOD: track 0.00 -> 1.92 mm
- net BCKOUT33: track 7.05 -> 8.81 mm
- net /ILIM: track 1.63 -> 0.00 mm
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Other:
- board outline added: 7.8 x 88.3 mm
- board text added: "Sig G Sig Pow G Sig"
- board text removed: "Sig G Sig Pow G S"

Commit message: application
Parts:
- added H1: ~, MountingHole:MountingHole_2.5mm, F.Cu at (89.0, 143.8)
- added H2: ~, MountingHole:MountingHole_2.5mm, F.Cu at (161.6, 87.4)
- added H3: ~, MountingHole:MountingHole_2.5mm, F.Cu at (161.6, 133.8)
- CON1: moved to B.Cu
- SW3, SW4: footprint fpl:SW-TH_5P-L6.0-W6.0-P4.50-LS6.5 -> fpl:KEY-SMD_4P-L6.0-W6.0-P4.50-LS10.0
- moved D2 178.3 mm to (83.3, 102.7), turned to 180 degrees
- moved D1 166.8 mm to (97.1, 104.2), turned to 90 degrees
- moved R3 163.3 mm to (97.1, 107.8), turned to 90 degrees
- moved R16 136.0 mm to (86.5, 102.7)
- moved D3 132.1 mm to (129.8, 103.4)
- moved NT1 128.1 mm to (162.6, 16.9), turned to 90 degrees
- moved BZ1 111.5 mm to (154.6, 112.2)
- moved J5 111.0 mm to (147.0, 134.6), turned to 90 degrees
- moved J4 108.8 mm to (144.0, 134.6), turned to 90 degrees
- moved J3 106.6 mm to (141.0, 134.6), turned to 90 degrees
- moved C20 105.1 mm to (109.7, 145.3), turned to 90 degrees
- moved J2 104.6 mm to (138.0, 134.6), turned to 90 degrees
- moved J1 102.7 mm to (135.0, 134.6), turned to 90 degrees
- moved NT2 97.5 mm to (149.7, 8.24), turned to 90 degrees
- moved NT3 96.2 mm to (151.2, 8.24), turned to 90 degrees
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Connections:
- U6 pad 12: GNDD -> (no net)
- U6 pad 13: GNDD -> (no net)
- U6 pad 14: GNDD -> (no net)
- U6 pad 15: GNDD -> (no net)
Other:
- board size 7.8 x 88.3 mm -> 104.3 x 85.8 mm
- board text added: "3.3V"
- board text added: "5V"
- board text added: "ESP32 USB"
- board text added: "STM32 USB"
- board text added: "VB"

Commit message: application
Parts:
- moved C20 75.1 mm to (163.1, 92.5)
- moved R14 43.9 mm to (112.0, 102.0), turned to 180 degrees
- moved R15 43.7 mm to (109.0, 102.0), turned to 180 degrees
- moved NT1 40.0 mm to (171.4, 56.0)
- moved NT2 40.0 mm to (158.5, 47.3)
- moved NT3 40.0 mm to (160.0, 47.3)
- moved R24 31.3 mm to (142.0, 106.6), turned to -90 degrees
- moved R27 30.9 mm to (144.6, 106.6)
- moved D6 30.6 mm to (144.6, 103.2)
- moved D5 30.6 mm to (142.0, 103.2), turned to -90 degrees
- moved Q3 20.1 mm to (154.3, 105.2), turned to 90 degrees
- moved SW5 19.3 mm to (132.9, 130.0), turned to -45 degrees
- moved R42 17.5 mm to (157.3, 107.0), turned to -90 degrees
- moved R48 13.7 mm to (154.3, 108.4), turned to 0 degrees
- moved SW2 11.1 mm to (125.1, 122.2), turned to -45 degrees
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Routing:
- net /VDDASTM: track 3.59 -> 1.40 mm
- net VDD: vias 2 -> 1
- net GNDHSC: vias 29 -> 36
Other:
- board size 104.3 x 85.8 mm -> 91.4 x 55.4 mm
