File: device/hw/$pr/medmentum.kicad_pcb (KiCad board)
At the start: 6 copper layers, 91.4 x 55.4 mm, 134 parts, among them CON1 ZX-IDC2.54-2-13PZZ, J1 Conn_01x01_Pin, J2 Conn_01x01_Pin, J3 Conn_01x01_Pin, J4 Conn_01x01_Pin, J5 Conn_01x01_Pin, Q1 PNP, Q2 NPN, Q3 NPN, SW1 SW_SPDT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

Commit message: application
Parts:
- added G***: LOGO, LOGO, F.Cu at (100.2, 105.8)
- added G***: LOGO, LOGO, F.Cu at (131.3, 106.8)
- added G***: LOGO, LOGO, F.Cu at (105.7, 105.8)
- added G***: LOGO, LOGO, F.Cu at (94.7, 105.8)
- added G***: LOGO, LOGO, F.Cu at (85.0, 105.9)
- moved R45 47.0 mm to (123.4, 103.7)
- moved R51 41.9 mm to (128.3, 112.2)
- moved H1 39.4 mm to (75.8, 106.7)
- moved TH1 35.9 mm to (118.1, 97.5)
- moved NT1 35.6 mm to (183.5, 89.5)
- moved NT2 35.6 mm to (170.6, 80.8)
- moved NT3 35.6 mm to (172.1, 80.8)
- moved R49 12.7 mm to (133.6, 112.5)
- moved C36 12.7 mm to (132.0, 112.4)
- moved C1 8.74 mm to (91.4, 95.5)
- moved R28 8.01 mm to (108.3, 102.2), turned to -90 degrees
- moved R18 7.47 mm to (102.8, 102.2), turned to -90 degrees
- moved R3 7.18 mm to (97.3, 102.2), turned to -90 degrees
- moved C20 4.26 mm to (162.4, 96.7)
- moved D7 3.50 mm to (108.3, 105.8), turned to -90 degrees
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Connections:
- CON1 pad 14: /CONFSW_DB -> /CONFSW
- CON1 pad 16: /HOSW_DB -> /HOSW
- U7 pad 41: /CONFSW -> /CONFSW_DB
- U7 pad 45: /HOSW -> /HOSW_DB
Routing:
- net VBUS: track 0.97 -> 30.7 mm, vias 4 -> 5
- net GNDD: track 11.8 -> 29.7 mm, vias 8 -> 14
- net /UARTRX_ESP: track 0.00 -> 10.8 mm, vias 0 -> 2
- net /UARTTX_ESP: track 0.00 -> 9.33 mm, vias 0 -> 2
- net BATSYS: track 13.6 -> 5.48 mm
- net BCKOUT5: track 5.83 -> 11.0 mm
- net BCOUT: track 17.6 -> 13.3 mm
- net Net-(U8-IO2): track 0.00 -> 3.45 mm
- net /ENRST: track 0.00 -> 3.34 mm
- net BCKOUT33: track 8.81 -> 11.3 mm, vias 0 -> 1
- net Net-(U8-IO9): track 0.00 -> 2.11 mm
- net /ITERM: track 2.03 -> 0.00 mm
- net Net-(D7-K): track 0.00 -> 1.86 mm
- net Net-(D4-K): track 0.00 -> 1.84 mm
- net Net-(D1-K): track 0.00 -> 1.84 mm
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Other:
- board text added: "3V3"
- board text removed: "3.3V"

Commit message: application
Parts:
- removed G*** (x5): LOGO, LOGO
- C22: value 4.7u -> 1u; footprint Capacitor_SMD:C_0805_2012Metric -> Capacitor_SMD:C_0603_1608Metric
- TH1: moved to F.Cu
- moved C20 138.4 mm to (34.4, 44.0), turned to 0 degrees
- moved R42 133.7 mm to (50.4, 26.5), turned to 0 degrees
- moved C29 133.5 mm to (38.4, 29.0), turned to 0 degrees
- moved R47 128.7 mm to (50.4, 31.5), turned to 0 degrees
- moved R48 127.7 mm to (50.4, 34.0)
- moved C36 127.6 mm to (42.4, 21.4), turned to 0 degrees
- moved R24 124.8 mm to (46.4, 26.5), turned to 0 degrees
- moved R27 123.6 mm to (46.4, 31.5), turned to 0 degrees
- moved R50 123.2 mm to (50.4, 36.5), turned to 0 degrees
- moved D2 120.1 mm to (166.2, 12.8)
- moved R40 113.4 mm to (50.4, 24.0), turned to 0 degrees
- moved R32 112.2 mm to (46.4, 39.0)
- moved R17 111.2 mm to (42.4, 39.0)
- moved SW5 109.3 mm to (224.6, 70.5), turned to 90 degrees
- moved R51 106.9 mm to (50.4, 39.0), turned to 0 degrees
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Connections:
- C18 pad 2: GNDHSC -> GNDD
- C19 pad 1: GNDHSC -> GNDD
- R28 pad 1: GNDD -> LGND
- R3 pad 1: GNDD -> LGND
- U3 pad 1: /-USB_D -> /USB_D-
- U3 pad 3: /+USB_D -> /USB_D+
- USB1 pad 10: /+USB_D -> /USB_D+
- USB1 pad 7: /-USB_D -> /USB_D-
- USB1 pad 8: /+USB_D -> /USB_D+
- USB1 pad 9: /-USB_D -> /USB_D-
- Y2 pad 2: GNDHSC -> GNDD
- Y2 pad 4: GNDHSC -> GNDD
Routing:
- net VBUS: track 30.7 -> 7.81 mm, vias 5 -> 2
- net VDD: track 0.72 -> 18.5 mm, vias 1 -> 3
- net /BAT: track 13.5 -> 0.00 mm, vias 3 -> 0
- net BCOUT: track 13.3 -> 0.00 mm, vias 3 -> 0
- net BCKOUT5: track 11.0 -> 0.00 mm
- net /UARTRX_ESP: track 10.8 -> 0.00 mm, vias 2 -> 0
- net /UARTTX_ESP: track 9.33 -> 0.00 mm, vias 2 -> 0
- net BCKOUT33: track 11.3 -> 3.60 mm, vias 1 -> 5
- net /VDDASTM: track 1.40 -> 8.65 mm, vias 1 -> 0
- net GNDD: track 29.7 -> 22.7 mm, vias 14 -> 5
- net GNDA: track 1.00 -> 7.79 mm, vias 1 -> 3
- net /HSE_OUT: track 15.6 -> 9.94 mm
- net /USB_D+: track 2.04 -> 7.67 mm
- net BATSYS: track 5.48 -> 0.00 mm, vias 2 -> 0
- net /USB_D-: track 2.04 -> 7.49 mm
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Other:
- board size 91.4 x 55.4 mm -> 98 x 42.5 mm
- board text removed: "3V3"
- board text removed: "5V"
- board text removed: "ESP32 USB"
- board text removed: "STM32 USB"
- board text removed: "VB"

Commit message: application
Parts:
- removed NT2, NT3: NetTie_2, NetTie:NetTie-2_SMD_Pad0.5mm
- moved C20 167.6 mm to (193.6, 96.4), turned to 45 degrees
- moved C29 164.9 mm to (184.7, 105.1), turned to -135 degrees
- moved C35 155.3 mm to (179.8, 108.4), turned to -45 degrees
- moved R45 152.2 mm to (181.0, 107.2), turned to -45 degrees
- moved R40 151.1 mm to (176.5, 107.3), turned to -45 degrees
- moved C30 150.2 mm to (168.2, 106.9), turned to -135 degrees
- moved C33 148.1 mm to (169.4, 108.1), turned to -135 degrees
- moved C31 147.3 mm to (167.1, 105.8), turned to -135 degrees
- moved R32 145.4 mm to (174.3, 108.4), turned to -135 degrees
- moved C34 145.3 mm to (169.2, 104.6), turned to 135 degrees
- moved C32 143.4 mm to (166.2, 101.6), turned to -90 degrees
- moved R33 137.1 mm to (169.6, 101.7), turned to 180 degrees
- moved R34 135.3 mm to (169.6, 99.9), turned to 180 degrees
- moved C3 129.1 mm to (135.3, 104.5)
- moved C4 126.9 mm to (137.1, 100.9), turned to 90 degrees
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Connections:
- D8 pad 1: /SW_BOOT0 -> /SW_BOOTE0
- D9 pad 2: /SW_BOOT0 -> /SW_BOOTE0
- R14 pad 1: Net-(D2-A) -> Net-(R14-Pad1)
- R14 pad 2: Net-(R14-Pad2) -> /USB_SLC
- R15 pad 1: Net-(R14-Pad2) -> Net-(D2-A)
- R15 pad 2: /USB_SLC -> Net-(R14-Pad1)
- R43 pad 1: Net-(R43-Pad1) -> /SW_BOOTE0
- R43 pad 2: Net-(U8-IO9) -> Net-(R43-Pad2)
- R46 pad 1: /SW_BOOT0 -> Net-(R43-Pad2)
- R46 pad 2: Net-(R43-Pad1) -> Net-(U8-IO9)
- SW5 pad 2: /SW_BOOT0 -> /SW_BOOTE0
Routing:
- net /BAT: track 0.00 -> 21.5 mm, vias 0 -> 3
- net /UARTTX_ESP: track 0.00 -> 17.3 mm, vias 0 -> 2
- net /UARTRX_ESP: track 0.00 -> 16.8 mm, vias 0 -> 2
- net GNDD: track 22.7 -> 35.1 mm
- net BCKOUT33: track 3.60 -> 15.9 mm, vias 5 -> 6
- net BATSYS: track 0.00 -> 11.5 mm, vias 0 -> 2
- net VBUS: track 7.81 -> 16.7 mm
- net BCOUT: track 0.00 -> 8.74 mm, vias 0 -> 2
- net Net-(U8-IO2): track 0.00 -> 5.99 mm
- net LVCC: track 0.00 -> 4.70 mm
- net /BCK5_EN: track 0.00 -> 4.63 mm
- net /STM_UARTRX: track 1.02 -> 4.84 mm, vias 1 -> 0
- net /ITERM: track 0.00 -> 3.73 mm
- net /STM_UARTTX: track 0.71 -> 3.98 mm, vias 1 -> 0
- net /ENRST: track 0.00 -> 3.08 mm
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
Commit message: application
Parts:
- TH1: moved to B.Cu
- moved R47 94.5 mm to (195.0, 95.6), turned to 135 degrees
- moved R24 93.8 mm to (189.3, 101.3), turned to 135 degrees
- moved D5 91.2 mm to (188.0, 102.6), turned to -45 degrees
- moved D8 91.0 mm to (193.6, 97.0), turned to -45 degrees
- moved R50 90.2 mm to (190.7, 99.9), turned to -45 degrees
- moved R27 89.7 mm to (185.3, 105.1), turned to -45 degrees
- moved D6 89.4 mm to (186.6, 103.9), turned to 135 degrees
- moved D9 89.2 mm to (192.0, 98.5), turned to 135 degrees
- moved D1 87.5 mm to (102.3, 89.2), turned to 180 degrees
- moved R3 85.5 mm to (105.9, 89.2), turned to 180 degrees
- moved R17 79.5 mm to (170.7, 85.6)
- moved D3 66.3 mm to (167.5, 85.6)
- moved C36 64.0 mm to (152.0, 105.7), turned to 135 degrees
- moved R49 56.4 mm to (151.1, 106.7), turned to 135 degrees
- moved R51 52.9 mm to (153.2, 104.5), turned to 135 degrees
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Routing:
- net /SERVOPWM1: track 1.02 -> 43.7 mm
- net /FG_GPOUT: track 2.18 -> 44.9 mm
- net /SERVOPWM3: track 1.02 -> 42.8 mm
- net /SERVOPWM2: track 0.71 -> 39.0 mm
- net /SERVOPWM4: track 0.71 -> 38.0 mm
- net /USB_DSTM+: track 1.66 -> 38.8 mm
- net /USB_DSTM-: track 1.56 -> 38.0 mm
- net /CHG_#PGOOD: track 2.82 -> 34.8 mm, vias 1 -> 2
- net /BUZPWM: track 1.01 -> 32.4 mm
- net /CHG_#CHG: track 3.00 -> 34.0 mm, vias 1 -> 2
- net /SERVOPWM5: track 2.70 -> 29.2 mm
- net VBUS: track 16.7 -> 41.9 mm, vias 2 -> 3
- net /SERVOPWM6: track 1.80 -> 23.3 mm
- net /PANICGPIO: track 1.01 -> 22.2 mm
- net /USB_DESP+: track 1.26 -> 17.4 mm
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
Commit message: application
Parts:
- turned TH1 to 0 degrees
Routing:
- net /USB_SLC: track 0.45 -> 68.0 mm, vias 1 -> 2
- net /FG_SCL: track 3.79 -> 59.5 mm
- net Net-(U8-IO9): track 0.68 -> 55.6 mm
- net /FG_SDA: track 4.05 -> 50.9 mm
- net /LEDCHPWM: track 0.67 -> 28.0 mm, vias 1 -> 2
- net /IICDISP_SCL: track 1.97 -> 27.9 mm
- net /IICDISP_SDA: track 3.84 -> 25.0 mm
- net /PANICPWM: track 1.02 -> 17.8 mm
- net /TS: track 0.00 -> 16.1 mm, vias 0 -> 1
- net /BOOT0: track 1.02 -> 16.7 mm, vias 1 -> 3
- net /CONFSW_DB: track 0.00 -> 10.7 mm, vias 1 -> 2
- net /HOSW_DB: track 0.71 -> 7.28 mm, vias 1 -> 2
- net /BUZPWM: track 32.4 -> 34.3 mm
- net /SERVOPWM6: track 23.3 -> 22.1 mm
- net BCKOUT33: track 15.9 -> 16.6 mm
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
Commit message: application
Parts:
- moved R43 0.80 mm to (187.0, 86.8)
- moved R46 0.80 mm to (185.0, 88.8)
Routing:
- net /LEDHOPWM: track 0.75 -> 25.5 mm, vias 1 -> 2
- net /SERVOPWM5: track 29.0 -> 30.1 mm
- net Net-(U8-IO9): track 55.6 -> 56.4 mm, vias 1 -> 2
Changed lines of the file:
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@@
 	(footprint "Resistor_SMD:R_0402_1005Metric"
 		(layer "F.Cu")
-		(at 184.194376 88.589594 -135)
+		(at 184.9542 88.83377 -135)
 		(descr "Resistor SMD 0402 (1005 Metric), square (rectangular) end terminal, IPC_7351 nominal, (Body size source: IPC-SM-782 page 72, https://www.pcb-3d.com/wordpress/wp-content/uploads/ipc-sm-782a_amendment_1_and_2.pdf), generated with kicad-footprint-generator")
 		(tags "resistor")
@@
 	(footprint "Resistor_SMD:R_0805_2012Metric"
 		(layer "F.Cu")
-		(at 186.226376 86.557594 -135)
+		(at 186.9862 86.80177 -135)
 		(descr "Resistor SMD 0805 (2012 Metric), square (rectangular) end terminal, IPC_7351 nominal, (Body size source: IPC-SM-782 page 72, https://www.pcb-3d.com/wordpress/wp-content/uploads/ipc-sm-782a_amendment_1_and_2.pdf), generated with kicad-footprint-generator")
 		(tags "resistor")
@@
 	)
 	(via
-		(at 161.764 87.13197)
+		(at 162.018 86.87797)
 		(size 0.4)
 		(drill 0.2)
@@
 	)
 	(segment
-		(start 158.0192 83.38717)
-		(end 158.0192 82.96337)
+		(start 161.51 86.87797)
+		(end 158.0192 83.38717)
 		(width 0.2)
 		(layer "In2.Cu")
@@
 	)
 	(segment
-		(start 161.764 87.13197)
-		(end 158.0192 83.38717)
+		(start 162.018 86.87797)
+		(end 161.51 86.87797)
 		(width 0.2)
 		(layer "In2.Cu")
@@
 	)
 	(segment
-		(start 164.8628 107.41877)
-		(end 164.865 107.42097)
+		(start 158.0192 83.38717)
+		(end 158.0192 82.96337)
+		(width 0.2)
+		(layer "In2.Cu")
+		(net 24)
+	)
+	(segment
+		(start 162.018 86.87797)
+		(end 162.018 94.62497)
 		(width 0.2)
 		(layer "B.Cu")
@@
 	)
 	(segment
-		(start 161.764 94.37097)
-		(end 164.8628 97.46977)
+		(start 164.8628 107.41877)
+		(end 164.865 107.42097)
 		(width 0.2)
 		(layer "B.Cu")
@@
 	)
 	(segment
-		(start 161.764 87.13197)
-		(end 161.764 94.37097)
+		(start 162.018 94.62497)
+		(end 164.8628 97.46977)
 		(width 0.2)
 		(layer "B.Cu")
@@
 	)
 	(segment
-		(start 162.362 87.76697)
-		(end 162.362 88.01797)
-		(width 0.2)
-		(layer "F.Cu")
-		(net 26)
-	)
-	(segment
-		(start 161.064 89.31597)
+		(start 160.977 89.31597)
 		(end 160.585 89.31597)
 		(width 0.2)
@@
 	)
 	(segment
-		(start 162.362 88.01797)
-		(end 161.064 89.31597)
+		(start 162.907 87.38597)
+		(end 160.977 89.31597)
 		(width 0.2)
 		(layer "F.Cu")
@@
 	)
 	(via
-		(at 162.362 87.76697)
+		(at 162.907 87.38597)
 		(size 0.4)
 		(drill 0.2)
@@
 	)
 	(segment
-		(start 162.362 87.76697)
-		(end 162.362 94.33397)
+		(start 162.399 87.89397)
+		(end 162.399 94.37097)
 		(width 0.2)
 		(layer "B.Cu")
@@
 	)
 	(segment
-		(start 162.362 94.33397)
-		(end 171.289 103.26097)
+		(start 171.289 108.76497)
+		(end 172.485 109.96097)
 		(width 0.2)
 		(layer "B.Cu")
@@
 	)
 	(segment
-		(start 171.289 108.76497)
-		(end 172.485 109.96097)
+		(start 162.907 87.38597)
+		(end 162.399 87.89397)
+		(width 0.2)
+		(layer "B.Cu")
+		(net 26)
+	)
+	(segment
+		(start 162.399 94.37097)
+		(end 171.289 103.26097)
 		(width 0.2)
 		(layer "B.Cu")
@@
 	)
 	(segment
-		(start 161.256 87.63697)
-		(end 161.256 88.48897)
+		(start 161.256 87.89397)
+		(end 161.256 88.52897)
 		(width 0.2)
 		(layer "F.Cu")
@@
 	)
 	(segment
-		(start 160.929 88.81597)
-		(end 160.585 88.81597)
+		(start 161.129 87.76697)
+		(end 161.256 87.89397)
+		(width 0.2)
+		(layer "F.Cu")
+		(net 28)
+	)
+	(segment
+		(start 161.256 88.52897)
+		(end 160.969 88.81597)
 		(width 0.2)
 		(layer "F.Cu")
@@
 	)
 	(segment
-		(start 161.256 88.48897)
-		(end 160.929 88.81597)
+		(start 160.969 88.81597)
+		(end 160.585 88.81597)
 		(width 0.2)
 		(layer "F.Cu")
@@
 	)
 	(via
-		(at 161.256 87.63697)
+		(at 161.129 87.76697)
 		(size 0.4)
 		(drill 0.2)
@@
 	)
 	(segment
-		(start 161.256 105.94997)
-		(end 159.785 107.42097)
+		(start 161.256 87.89397)
+		(end 161.256 105.80097)
+		(width 0.2)
+		(layer "B.Cu")
+		(net 28)
+	)
+	(segment
+		(start 161.256 105.80097)
+		(end 159.785 107.27197)
+		(width 0.2)
+		(layer "B.Cu")
+		(net 28)
+	)
+	(segment
+		(start 161.129 87.76697)
+		(end 161.256 87.89397)
 		(width 0.2)
 		(layer "B.Cu")
@@
 	)
 	(segment
-		(start 161.256 87.63697)
-		(end 161.256 105.94997)
+		(start 159.785 107.27197)
+		(end 159.785 107.42097)
 		(width 0.2)
 		(layer "B.Cu")
@@
 	)
 	(via
+		(at 160.7226 84.97297)
+		(size 0.4)
+		(drill 0.2)
+		(layers "F.Cu" "B.Cu")
+		(net 32)
+	)
+	(via
 		(at 159.6956 83.80157)
 		(size 0.4)
@@
 	)
 	(segment
+		(start 160.7226 84.97297)
+		(end 159.6956 83.94597)
+		(width 0.2)
+		(layer "In2.Cu")
+		(net 32)
+	)
+	(segment
+		(start 159.6956 83.94597)
+		(end 159.6956 83.80157)
+		(width 0.2)
+		(layer "In2.Cu")
+		(net 32)
+	)
+	(segment
+		(start 161.637 87.25897)
+		(end 161.637 105.80097)
+		(width 0.2)
+		(layer "B.Cu")
+		(net 32)
+	)
+	(segment
+		(start 160.7226 86.34457)
+		(end 161.637 87.25897)
+		(width 0.2)
+		(layer "B.Cu")
+		(net 32)
+	)
+	(segment
+		(start 162.325 106.48897)
+		(end 162.325 107.42097)
+		(width 0.2)
+		(layer "B.Cu")
+		(net 32)
+	)
+	(segment
+		(start 161.637 105.80097)
+		(end 162.325 106.48897)
+		(width 0.2)
+		(layer "B.Cu")
+		(net 32)
+	)
+	(segment
+		(start 160.7226 84.97297)
+		(end 160.7226 86.34457)
+		(width 0.2)
+		(layer "B.Cu")
+		(net 32)
+	)
+	(segment
 		(start 152.7106 88.31597)
 		(end 153.725 88.31597)
@@
 		(net 82)
 	)
+	(via
+		(at 184.2938 89.49417)
+		(size 0.4)
+		(drill 0.2)
+		(layers "F.Cu" "B.Cu")
+		(net 82)
+	)
 	(segment
-		(start 170.781 82.30597)
-		(end 177.131 82.30597)
+		(start 184.2938 89.46877)
+		(end 184.2938 89.49417)
 		(width 0.2)
 		(layer "In2.Cu")
@@
 	)
 	(segment
-		(start 134.245 88.85917)
-		(end 134.7638 88.85917)
+		(start 141.317 82.30597)
+		(end 177.131 82.30597)
 		(width 0.2)
 		(layer "In2.Cu")
@@
 	(segment
 		(start 177.131 82.30597)
-		(end 183.735 88.90997)
+		(end 184.2938 89.46877)
 		(width 0.2)
 		(layer "In2.Cu")
@@
 	)
 	(segment
-		(start 141.317 82.30597)
-		(end 170.781 82.30597)
+		(start 134.7638 88.85917)
+		(end 141.317 82.30597)
 		(width 0.2)
 		(layer "In2.Cu")
@@
 	)
 	(segment
-		(start 134.7638 88.85917)
-		(end 141.317 82.30597)
+		(start 134.245 88.85917)
+		(end 134.7638 88.85917)
 		(width 0.2)
 		(layer "In2.Cu")

Commit message: application
Parts:
- turned C29 to 45 degrees
Routing:
- net Net-(D2-A): track 0.00 -> 78.0 mm, vias 0 -> 2
- net /ENRST: track 3.08 -> 29.1 mm
- net /NRST: track 4.04 -> 24.2 mm, vias 1 -> 2
- net Net-(BZ1--): track 0.00 -> 17.7 mm
- net BCKOUT5: track 2.91 -> 18.6 mm
- net GNDD: track 35.1 -> 44.3 mm
- net Net-(U7-PA14): track 0.71 -> 6.49 mm, vias 1 -> 2
- net /BUZPWM: vias 1 -> 2

Commit message: application
Parts:
- moved R3 0.06 mm to (105.8, 89.2)
Connections:
- BAT1 pad 2: GNDD -> BCKOUT33
- U7 pad 50: (no net) -> GNDD
Routing:
- net GNDD: track 44.3 -> 331.2 mm, vias 5 -> 28
- net BCKOUT5: track 18.6 -> 187.6 mm, vias 1 -> 5
- net BCKOUT33: track 16.7 -> 146.7 mm, vias 6 -> 17
- net LGND: track 0.00 -> 106.5 mm, vias 0 -> 4
- net VBUS: track 41.9 -> 123.6 mm, vias 3 -> 5
- net LVCC: track 4.70 -> 71.9 mm, vias 0 -> 4
- net BATSYS: track 11.5 -> 76.2 mm, vias 2 -> 3
- net GNDA: track 7.79 -> 60.7 mm
- net /CONFSW: track 0.00 -> 22.9 mm, vias 0 -> 1
- net BCOUT: track 8.91 -> 31.0 mm, vias 2 -> 4
- net /SW_BOOT0: track 0.00 -> 18.1 mm
- net /SW_BOOTE0: track 0.00 -> 16.9 mm
- net VDD: track 18.5 -> 33.8 mm
- net /HOSW: track 0.00 -> 14.5 mm, vias 0 -> 1
- net Net-(BZ1--): track 17.7 -> 24.9 mm
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- added copper zone on In3.Cu, net BCKOUT33
- added copper zone on In1.Cu, net GNDD
- added copper zone on In4.Cu, net GNDD
