File: device/hw/$pr/medmentum.kicad_pcb (KiCad board)
At the start: 6 copper layers, 98 x 42.5 mm, 132 parts, among them CON1 ZX-IDC2.54-2-13PZZ, J1 Conn_01x01_Pin, J2 Conn_01x01_Pin, J3 Conn_01x01_Pin, J4 Conn_01x01_Pin, J5 Conn_01x01_Pin, Q1 PNP, Q2 NPN, Q3 NPN, SW1 SW_SPDT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

Commit message: application
Connections:
- U4 pad 18: (no net) -> GNDD
- U6 pad 12: (no net) -> GNDD
- U6 pad 13: (no net) -> GNDD
- U6 pad 14: (no net) -> GNDD
- U6 pad 15: (no net) -> GNDD
Routing:
- net GNDD: track 331.2 -> 216.4 mm, vias 28 -> 29
- net BCKOUT33: track 146.7 -> 85.8 mm, vias 17 -> 18
- net VBUS: track 123.6 -> 105.9 mm
- net BCKOUT5: track 187.6 -> 175.0 mm
- net LGND: track 106.5 -> 101.2 mm
- net /ITERM: track 6.20 -> 4.96 mm
- net /LEDCHPWM: track 28.9 -> 27.8 mm
- net GNDA: track 60.7 -> 61.5 mm

Commit message: application
Routing:
- net GNDD: track 216.4 -> 174.3 mm, vias 29 -> 107
- net BCKOUT33: track 85.8 -> 73.2 mm, vias 18 -> 20
- net VBUS: track 105.9 -> 103.0 mm
- net Net-(D2-A): track 77.1 -> 74.5 mm
- net BCKOUT5: track 175.0 -> 174.1 mm
- net /LEDCHPWM: track 27.8 -> 28.6 mm
- net /FG_SDA: vias 2 -> 3

Commit message: application
Parts:
- added G***: LOGO, LOGO, B.Cu at (116.8, 115.1)
- added G***: LOGO, LOGO, B.Cu at (111.0, 109.3)
Connections:
- BAT1 pad 2: BCKOUT33 -> GNDD
Routing:
- net GNDD: track 174.3 -> 169.5 mm, vias 107 -> 127
- net BCKOUT33: track 73.2 -> 70.8 mm
- net LGND: track 101.2 -> 100.5 mm
- net LVCC: track 72.2 -> 71.7 mm
Other:
- board text added: "MEDMENTUM"
- board text added: "Ognjen Guteša T31 Uz podršku mentora Novice Gutovića i odeljenskog starešine Aleksandre Rakić Todorović."
- board text removed: "Sig G Sig Pow G Sig"

Commit message: application
Parts:
- moved C3 0.16 mm to (115.0, 96.3)
Routing:
- net GNDD: track 169.5 -> 146.1 mm, vias 127 -> 190
- net /USB_D-: track 12.8 -> 7.84 mm
- net Net-(BZ1--): track 24.9 -> 20.1 mm
- net BCOUT: track 31.0 -> 27.3 mm
- net /USB_D+: track 10.5 -> 8.14 mm
- net LGND: track 100.5 -> 102.8 mm, vias 4 -> 5
- net BCKOUT33: track 70.8 -> 68.7 mm
- net /ENRST: track 31.7 -> 33.1 mm
- net /FG_SDA: vias 3 -> 2
- added copper zone on F.Cu, net GNDD
