File: device/hw/$pr/Sheets/north_bridge.kicad_sch (KiCad schematic)
At the start: 0 parts

Commit message: BMS
Other:
- company: (none) -> ETŠ Mihajlo Pupin "Medmentum"
Changed lines of the file:
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@@
 	(generator_version "8.0")
 	(paper "A4")
+	(title_block
+		(company "ETŠ Mihajlo Pupin \"Medmentum\"")
+	)
 	(sheet
 		(at 81.28 68.58)
