File: device/hw/$pr/Sheets/peripherals.kicad_sch (KiCad schematic)
At the start: 0 parts

Commit message: BMS
Other:
- company: (none) -> ETŠ Mihajlo Pupin "Medmentum"
Changed lines of the file:
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@@
 	(generator_version "8.0")
 	(paper "A4")
+	(title_block
+		(company "ETŠ Mihajlo Pupin \"Medmentum\"")
+	)
 	(sheet
 		(at 74.93 40.64)

Commit message: application
Other:
- removed sheet Biometric
- removed sheet Touch
Changed lines of the file:
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@@
-	)
-	(sheet
-		(at 25.4 33.02)
-		(size 24.13 13.97)
-		(fields_autoplaced yes)
-		(stroke
-			(width 0.1524)
-			(type solid)
-		)
-		(fill
-			(color 0 0 0 0.0000)
-		)
-		(property "Sheetname" "Touch"
-			(at 25.4 32.3084 0)
-			(effects
-				(font
-					(size 1.27 1.27)
-				)
-				(justify left bottom)
-			)
-		)
-		(property "Sheetfile" "Peripherals/touch.kicad_sch"
-			(at 25.4 47.5746 0)
-			(effects
-				(font
-					(size 1.27 1.27)
-				)
-				(justify left top)
-			)
-		)
-		(instances
-			(project "medmentum"
-				(path "/ead52261-b3da-41ef-908f-3daaabe10954/df886fcf-452c-4fb9-a819-05e60426a5e4"
-					(page "8")
-				)
-			)
-		)
-	)
-	(sheet
-		(at 76.2 78.74)
-		(size 27.94 17.78)
-		(fields_autoplaced yes)
-		(stroke
-			(width 0.1524)
-			(type solid)
-		)
-		(fill
-			(color 0 0 0 0.0000)
-		)
-		(property "Sheetname" "Biometric"
-			(at 76.2 78.0284 0)
-			(effects
-				(font
-					(size 1.27 1.27)
-				)
-				(justify left bottom)
-			)
-		)
-		(property "Sheetfile" "Peripherals/biometric.kicad_sch"
-			(at 76.2 97.1046 0)
-			(effects
-				(font
-					(size 1.27 1.27)
-				)
-				(justify left top)
-			)
-		)
-		(instances
-			(project "medmentum"
-				(path "/ead52261-b3da-41ef-908f-3daaabe10954/df886fcf-452c-4fb9-a819-05e60426a5e4"
-					(page "12")
-				)
-			)
-		)
 	)
 	(sheet

Commit message: application
Parts:
- added BZ1: Buzzer, symbol Device:Buzzer
- added CON1: ZX-IDC2.54-2-13PZZ, fpl:IDC-TH_26P-P2.54_ZX-IDC2.54-2-13PZZ, symbol syl:ZX-IDC2.54-2-13PZZ
- added Q1: NPN, Package_TO_SOT_SMD:SOT-23, symbol Simulation_SPICE:NPN
- added R33: 1k, Resistor_SMD:R_2512_6332Metric, symbol Device:R_Small
- added R34: 1k, Resistor_SMD:R_2512_6332Metric, symbol Device:R
Connections:
- new net: BZ1.2 (-), Q1.1 (C), R33.1
- new net: Q1.2 (B), R34.2
- new net BCKOUT33: CON1.20, CON1.21, CON1.24, CON1.25
- new net BCKOUT5: CON1.12, CON1.13, CON1.2, CON1.4
- new net BUZPWM: R34.1
- new net BUZVCC: BZ1.1 (+), R33.2
- new net CONFSW: CON1.22
- new net GNDD: CON1.14, CON1.15, CON1.6, CON1.8, Q1.3 (E)
- new net HOSW: CON1.26
- new net IICDISP_SCL: CON1.9
- new net IICDISP_SDA: CON1.11
- new net LEDCHPWM: CON1.19
- new net LEDHOPWM: CON1.23
- new net PANICGPIO: CON1.17
- new net PANICPWM1: CON1.18
- new net PANICPWM2: CON1.16
- new net SERVOPWM1: CON1.1
- new net SERVOPWM2: CON1.3
- new net SERVOPWM3: CON1.5
- new net SERVOPWM4: CON1.7
- new net SERVOPWM5: CON1.10
Other:
- removed sheet Display
- removed sheet Motor
- removed sheet Speaker

Commit message: application
Parts:
- renumbered Q1 to Q3, R34 to R47, R33 to R48
Changed lines of the file:
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@@
 		(dnp no)
 		(fields_autoplaced yes)
-		(property "Reference" "Q1"
+		(property "Reference" "Q3"
 			(at 58.42 45.7199 0)
 			(effects
@@
 			(project "medmentum"
 				(path "/ead52261-b3da-41ef-908f-3daaabe10954/df886fcf-452c-4fb9-a819-05e60426a5e4"
-					(reference "Q1")
+					(reference "Q3")
 					(unit 1)
 				)
@@
 		(dnp no)
 		(fields_autoplaced yes)
-		(property "Reference" "#PWR084"
+		(property "Reference" "#PWR093"
 			(at 99.06 41.91 0)
 			(effects
@@
 			(project "medmentum"
 				(path "/ead52261-b3da-41ef-908f-3daaabe10954/df886fcf-452c-4fb9-a819-05e60426a5e4"
-					(reference "#PWR084")
+					(reference "#PWR093")
 					(unit 1)
 				)
@@
 		(on_board yes)
 		(dnp no)
-		(property "Reference" "R33"
+		(property "Reference" "R48"
 			(at 50.038 34.798 0)
 			(effects
@@
 			(project "medmentum"
 				(path "/ead52261-b3da-41ef-908f-3daaabe10954/df886fcf-452c-4fb9-a819-05e60426a5e4"
-					(reference "R33")
+					(reference "R48")
 					(unit 1)
 				)
@@
 		(dnp no)
 		(fields_autoplaced yes)
-		(property "Reference" "#PWR079"
+		(property "Reference" "#PWR097"
 			(at 106.68 26.67 0)
 			(effects
@@
 			(project "medmentum"
 				(path "/ead52261-b3da-41ef-908f-3daaabe10954/df886fcf-452c-4fb9-a819-05e60426a5e4"
-					(reference "#PWR079")
+					(reference "#PWR097")
 					(unit 1)
 				)
@@
 		(on_board yes)
 		(dnp no)
-		(property "Reference" "R34"
+		(property "Reference" "R47"
 			(at 39.37 43.688 90)
 			(effects
@@
 			(project "medmentum"
 				(path "/ead52261-b3da-41ef-908f-3daaabe10954/df886fcf-452c-4fb9-a819-05e60426a5e4"
-					(reference "R34")
+					(reference "R47")
 					(unit 1)
 				)
@@
 		(on_board yes)
 		(dnp no)
-		(property "Reference" "#PWR087"
+		(property "Reference" "#PWR0103"
 			(at 106.68 49.53 0)
 			(effects
@@
 			(project "medmentum"
 				(path "/ead52261-b3da-41ef-908f-3daaabe10954/df886fcf-452c-4fb9-a819-05e60426a5e4"
-					(reference "#PWR087")
+					(reference "#PWR0103")
 					(unit 1)
 				)
@@
 		(dnp no)
 		(fields_autoplaced yes)
-		(property "Reference" "#PWR088"
+		(property "Reference" "#PWR092"
 			(at 55.88 58.42 0)
 			(effects
@@
 			(project "medmentum"
 				(path "/ead52261-b3da-41ef-908f-3daaabe10954/df886fcf-452c-4fb9-a819-05e60426a5e4"
-					(reference "#PWR088")
+					(reference "#PWR092")
 					(unit 1)
 				)
@@
 		(on_board yes)
 		(dnp no)
-		(property "Reference" "#PWR090"
+		(property "Reference" "#PWR0104"
 			(at 106.68 54.61 0)
 			(effects
@@
 			(project "medmentum"
 				(path "/ead52261-b3da-41ef-908f-3daaabe10954/df886fcf-452c-4fb9-a819-05e60426a5e4"
-					(reference "#PWR090")
+					(reference "#PWR0104")
 					(unit 1)
 				)
@@
 		(dnp no)
 		(fields_autoplaced yes)
-		(property "Reference" "#PWR086"
+		(property "Reference" "#PWR094"
 			(at 88.9 44.45 0)
 			(effects
@@
 			(project "medmentum"
 				(path "/ead52261-b3da-41ef-908f-3daaabe10954/df886fcf-452c-4fb9-a819-05e60426a5e4"
-					(reference "#PWR086")
+					(reference "#PWR094")
 					(unit 1)
 				)
@@
 		(dnp no)
 		(fields_autoplaced yes)
-		(property "Reference" "#PWR085"
+		(property "Reference" "#PWR0102"
 			(at 116.84 41.91 0)
 			(effects
@@
 			(project "medmentum"
 				(path "/ead52261-b3da-41ef-908f-3daaabe10954/df886fcf-452c-4fb9-a819-05e60426a5e4"
-					(reference "#PWR085")
+					(reference "#PWR0102")
 					(unit 1)
 				)
@@
 		(dnp no)
 		(fields_autoplaced yes)
-		(property "Reference" "#PWR082"
+		(property "Reference" "#PWR0100"
 			(at 116.84 34.29 0)
 			(effects
@@
 			(project "medmentum"
 				(path "/ead52261-b3da-41ef-908f-3daaabe10954/df886fcf-452c-4fb9-a819-05e60426a5e4"
-					(reference "#PWR082")
+					(reference "#PWR0100")
 					(unit 1)
 				)
@@
 		(on_board yes)
 		(dnp no)
-		(property "Reference" "#PWR089"
+		(property "Reference" "#PWR096"
 			(at 99.06 57.15 0)
 			(effects
@@
 			(project "medmentum"
 				(path "/ead52261-b3da-41ef-908f-3daaabe10954/df886fcf-452c-4fb9-a819-05e60426a5e4"
-					(reference "#PWR089")
+					(reference "#PWR096")
 					(unit 1)
 				)
@@
 		(dnp no)
 		(fields_autoplaced yes)
-		(property "Reference" "#PWR080"
+		(property "Reference" "#PWR098"
 			(at 106.68 29.21 0)
 			(effects
@@
 			(project "medmentum"
 				(path "/ead52261-b3da-41ef-908f-3daaabe10954/df886fcf-452c-4fb9-a819-05e60426a5e4"
-					(reference "#PWR080")
+					(reference "#PWR098")
 					(unit 1)
 				)
@@
 		(dnp no)
 		(fields_autoplaced yes)
-		(property "Reference" "#PWR083"
+		(property "Reference" "#PWR0101"
 			(at 106.68 39.37 0)
 			(effects
@@
 			(project "medmentum"
 				(path "/ead52261-b3da-41ef-908f-3daaabe10954/df886fcf-452c-4fb9-a819-05e60426a5e4"
-					(reference "#PWR083")
+					(reference "#PWR0101")
 					(unit 1)
 				)
@@
 		(on_board yes)
 		(dnp no)
-		(property "Reference" "#PWR054"
+		(property "Reference" "#PWR095"
 			(at 99.06 52.07 0)
 			(effects
@@
 			(project "medmentum"
 				(path "/ead52261-b3da-41ef-908f-3daaabe10954/df886fcf-452c-4fb9-a819-05e60426a5e4"
-					(reference "#PWR054")
+					(reference "#PWR095")
 					(unit 1)
 				)
@@
 		(dnp no)
 		(fields_autoplaced yes)
-		(property "Reference" "#PWR081"
+		(property "Reference" "#PWR099"
 			(at 116.84 31.75 0)
 			(effects
@@
 			(project "medmentum"
 				(path "/ead52261-b3da-41ef-908f-3daaabe10954/df886fcf-452c-4fb9-a819-05e60426a5e4"
-					(reference "#PWR081")
-					(unit 1)
-				)
+					(reference "#PWR099")
+					(unit 1)
+				)
