File: device/hw/$pr/Sheets/Peripherals/motor.kicad_sch (KiCad schematic)
At the start: 0 parts

Commit message: BMS
Other:
- company: (none) -> ETŠ Mihajlo Pupin "Medmentum"
Changed lines of the file:
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@@
 	(generator_version "8.0")
 	(paper "A4")
+	(title_block
+		(company "ETŠ Mihajlo Pupin \"Medmentum\"")
+	)
 )

Commit message: application
Parts:
- added CON1: ZX-IDC2.54-2-10PZZ, fpl:IDC-TH_20P-P2.54_ZX-IDC2.54-2-10PZZ, symbol syl:ZX-IDC2.54-2-10PZZ
Changed lines of the file:
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@@
 		(company "ETŠ Mihajlo Pupin \"Medmentum\"")
 	)
+	(symbol
+		(lib_id "syl:ZX-IDC2.54-2-10PZZ")
+		(at 105.41 87.63 0)
+		(unit 1)
+		(exclude_from_sim no)
+		(in_bom yes)
+		(on_board yes)
+		(dnp no)
+		(property "Reference" "CON1"
+			(at 105.41 69.596 0)
+			(effects
+				(font
+					(size 1.27 1.27)
+				)
+			)
+		)
+		(property "Value" "ZX-IDC2.54-2-10PZZ"
+			(at 105.41 72.136 0)
+			(effects
+				(font
+					(size 1.27 1.27)
+				)
+			)
+		)
+		(property "Footprint" "fpl:IDC-TH_20P-P2.54_ZX-IDC2.54-2-10PZZ"
+			(at 105.41 106.68 0)
+			(effects
+				(font
+					(size 1.27 1.27)
+				)
+				(hide yes)
+			)
+		)
+		(property "Datasheet" ""
+			(at 105.41 87.63 0)
+			(effects
+				(font
+					(size 1.27 1.27)
+				)
+				(hide yes)
+			)
+		)
+		(property "Description" ""
+			(at 105.41 87.63 0)
+			(effects
+				(font
+					(size 1.27 1.27)
+				)
+				(hide yes)
+			)
+		)
+		(property "Package" "THT"
+			(at 105.41 68.58 0)
+			(effects
+				(font
+					(size 1.27 1.27)
+				)
+				(hide yes)
+			)
+		)
+		(property "MP" "ZX-IDC2.54-2-10PZZ"
+			(at 105.41 71.12 0)
+			(effects
+				(font
+					(size 1.27 1.27)
+				)
+				(hide yes)
+			)
+		)
+		(property "LCSCPart" "C7501245"
+			(at 105.41 109.22 0)
+			(effects
+				(font
+					(size 1.27 1.27)
+				)
+				(hide yes)
+			)
+		)
+		(pin "7"
+		)
+		(pin "6"
+		)
+		(pin "11"
+		)
+		(pin "14"
+		)
+		(pin "19"
+		)
+		(pin "16"
+		)
+		(pin "3"
+		)
+		(pin "2"
+		)
+		(pin "4"
+		)
+		(pin "20"
+		)
+		(pin "17"
+		)
+		(pin "9"
+		)
+		(pin "18"
+		)
+		(pin "8"
+		)
+		(pin "5"
+		)
+		(pin "12"
+		)
+		(pin "1"
+		)
+		(pin "10"
+		)
+		(pin "15"
+		)
+		(pin "13"
+		)
+		(instances
+			(project ""
+				(path "/ead52261-b3da-41ef-908f-3daaabe10954/df886fcf-452c-4fb9-a819-05e60426a5e4/84a05324-89a9-4757-ad4d-e9c84d1c42a7"
+					(reference "CON1")
+					(unit 1)
+				)
+			)
+		)
+	)
 )
