File: device/hw/$pr/Sheets/Peripherals/speaker.kicad_sch (KiCad schematic)
At the start: 0 parts

Commit message: BMS
Other:
- company: (none) -> ETŠ Mihajlo Pupin "Medmentum"
Changed lines of the file:
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@@
 	(generator_version "8.0")
 	(paper "A4")
+	(title_block
+		(company "ETŠ Mihajlo Pupin \"Medmentum\"")
+	)
 )

Commit message: application
Parts:
- added BZ1: Buzzer, symbol Device:Buzzer
- added Q1: NPN, symbol Simulation_SPICE:NPN
- added R28: 1k, symbol Device:R_Small
- added R29: 1k, symbol Device:R
Connections:
- new net: BZ1.2 (-), Q1.1 (C), R28.1
- new net: Q1.2 (B), R29.2
- new net BUZPWM: R29.1
- new net BUZVCC: BZ1.1 (+), R28.2
- new net GNDD: Q1.3 (E)

Commit message: application
Changed lines of the file:
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@@
 	(label "BUZPWM"
 		(at 120.65 107.95 0)
-		(fields_autoplaced yes)
 		(effects
 			(font
@@
 	(label "BUZVCC"
 		(at 144.78 90.17 90)
-		(fields_autoplaced yes)
 		(effects
 			(font
@@
 		)
 	)
+	(hierarchical_label "BUZPWM"
+		(shape input)
+		(at 119.38 107.95 180)
+		(effects
+			(font
+				(size 0.635 0.635)
+			)
+			(justify right)
+		)
+	)
