File: device/hw/$pr/Sheets/South Bridge/_autosave-bms.kicad_sch (KiCad schematic)
At the start: 21 parts, among them U1 BQ27441DRZR-G1B, U2 BQ24074RGTR

Commit message: application
Connections:
- net FG_GPOUT renamed SCL
- net FG_SDA renamed SDA
Changed lines of the file:
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@@
+		)
+	)
+	(text_box "Vin=0 VBAT=BAT"
+		(exclude_from_sim no)
+		(at 83.82 29.845 0)
+		(size 8.255 1.27)
+		(stroke
+			(width 0)
+			(type default)
+		)
+		(fill
+			(type none)
+		)
+		(effects
+			(font
+				(size 0.508 0.508)
+			)
+			(justify left top)
 		)
 	)
@@
 		)
 	)
+	(hierarchical_label "SCL"
+		(shape input)
+		(at 115.57 35.56 180)
+		(fields_autoplaced yes)
+		(effects
+			(font
+				(size 0.762 0.762)
+			)
+			(justify right)
+		)
+	)
+	(hierarchical_label "SDA"
+		(shape bidirectional)
+		(at 115.57 38.1 180)
+		(fields_autoplaced yes)
+		(effects
+			(font
+				(size 0.762 0.762)
+			)
+			(justify right)
+		)
+	)
