File: device/hw/$pr/Sheets/South Bridge/bms.kicad_sch (KiCad schematic)
At the start: 32 parts, among them U1 BQ27441DRZR-G1B, U2 BQ24074RGTR, U3 TPS63002DRCT, U4 TPS62082DSGR

Commit message: New-Sheet
Parts:
- added R15, R16: 5.1k 1%, symbol Device:R
- added USB1: USB-310F-B-SU, fpl:USB-310F-B-SU, symbol syl:USB-310F-B-SU
Connections:
- net GND: now also R15.2, R16.2, USB1.1 (GND), USB1.15 (GND), USB1.16 (GND), USB1.2 (GND)
- net VBUS: now also USB1.13 (VBUS), USB1.14 (VBUS), USB1.3 (VBUS), USB1.4 (VBUS)
- new net +USB_D: USB1.10 (D+), USB1.8 (D+)
- new net -USB_D: USB1.7 (D-), USB1.9 (D-)
- new net CC1: R15.1, USB1.6 (CC1)
- new net CC2: R16.1, USB1.12 (CC2)
- no-connect marks 2 -> 5
Other:
- note added: "Povuci D+ na 3.3V? Proveriti da li to MCU vec radi!"
- note added: "USB-C Connector"
- moved on the sheet: BAT, C1, C10, C2, C3, C4, C5, C6, C7, C8, C9, L1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
