File: device/hw/$pr/Sheets/South Bridge/bms.kicad_sch (KiCad schematic)
At the start: 21 parts, among them U1 BQ27441DRZR-G1B, U2 BQ24074RGTR

Commit message: application
Parts:
- added C10, C8, C9: 22u, symbol Device:C
- added C5, C6: 10u, symbol Device:C
- added C7: 100n, symbol Device:C
- added L1: 2.2uH, symbol Device:L
- added R14: 1M, symbol Device:R
- added R15: 1.6M, symbol Device:R
- added R16: 180k, symbol Device:R
- added U3: TPS63020DSJR, fpl:TPS63020DSJR, symbol syl:TPS63020DSJR
Connections:
- net BCOUT: now also C5.2, C6.2, U3.10 (VIN), U3.11 (VIN_11)
- net GNDD: now also C10.1, C5.1, C6.1, C7.1, C8.1, C9.1, R16.1, U3.15 (PGND), U3.2 (GND)
- net FG_GPOUT renamed SCL
- net FG_SDA renamed SDA
- new net: C7.2, U3.1 (VINA), U3.12 (EN), U3.13 (PS/SYNC)
- new net: R14.1, U3.14 (PG)
- new net: R15.1, R16.2, U3.3 (FB)
- new net: L1.2, U3.6 (L2), U3.7 (L2_7)
- new net: L1.1, U3.8 (L1), U3.9 (L1_9)
- new net BCKOUT: C10.2, C8.2, C9.2, R14.2, R15.2, U3.4 (VOUT), U3.5 (VOUT)

Commit message: application
Parts:
- L1: value 2.2uH -> 1.5uH
Other:
- note added: "Buck-Boost Converter"
- moved on the sheet: C10, C5, C6, C7, C8, C9, L1, R14, R15, R16, U3

Commit message: application
Parts:
- added C11: 10u, symbol Device:C
- added C12: 22u, symbol Device:C
- added L2: 1u, symbol Device:L
- added U4: TPS62082DSGR, fpl:TPS62082DSGR, symbol syl:TPS62082DSGR
Connections:
- net +BATT renamed BAT
- net BCKOUT renamed BCKOUT5
- net BCKOUT5: now also C11.2, U4.1 (EN), U4.8 (VIN)
- net GNDD renamed GND
- net GND: now also C11.1, C12.1, U4.2 (GND), U4.3 (MODE), U4.9 (GND), U4.9_1 (GND), U4.9_2 (GND)
- new net: L2.1, U4.7 (SW)
- new net BCKOUT33: C12.2, L2.2, U4.5 (VOS)
- no-connect marks 0 -> 2
Other:
- note added: "Buck-StepDown Fixed 3.3 Converter"
- moved on the sheet: BAT, C3, C4, R10, R4, R5, R6, R7, R8, R9, U1

Commit message: application
Parts:
- removed C10, C9: 22u, symbol Device:C
- removed R15: 1.6M, symbol Device:R
- removed R16: 180k, symbol Device:R
- removed U3: TPS63020DSJR, fpl:TPS63020DSJR, symbol syl:TPS63020DSJR
- added U3: TPS63002DRCT, fpl:TPS63002DRCR, symbol syl:TPS63002DRCT
- C6: value 10u -> 100n
- C7: value 100n -> 10u
- C8: value 22u -> 10u
- L1: value 1.5uH -> 2.2u
- R14: value 1M -> 100
- renumbered C12 to C10, C11 to C9
Connections:
- net BCKOUT5: now also C7.2, U3.1 (VOUT), U3.10 (FB); no longer R14.2
- net BCOUT: now also R14.2, U3.5 (VIN); no longer C6.2
- net GND: now also U3.11 (PP), U3.3 (PGND), U3.9 (GND)
- net at R14.1: now also C6.2, U3.6 (EN), U3.7 (PS/SYNC), U3.8 (VINA)
- net at L1.2: now also U3.2 (L2)
- net at L1.1: now also U3.4 (L1)
Other:
- note added: "!Mora biti blizu BAT!"
- moved on the sheet: BAT, C1, C10, C2, C3, C4, C9, L2, R1, R10, R11, R12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

Commit message: application
Parts:
- added R15, R16: 5.1k 1%, symbol Device:R
- added USB1: USB-310F-B-SU, fpl:USB-310F-B-SU, symbol syl:USB-310F-B-SU
Connections:
- net GND: now also R15.2, R16.2, USB1.1 (GND), USB1.15 (GND), USB1.16 (GND), USB1.2 (GND)
- net VBUS: now also USB1.13 (VBUS), USB1.14 (VBUS), USB1.3 (VBUS), USB1.4 (VBUS)
- new net +USB_D: USB1.10 (D+), USB1.8 (D+)
- new net -USB_D: USB1.7 (D-), USB1.9 (D-)
- new net CC1: R15.1, USB1.6 (CC1)
- new net CC2: R16.1, USB1.12 (CC2)
- no-connect marks 2 -> 5
Other:
- note added: "Buck-Boost Fixed 5V Converter"
- note added: "Povuci D+ na 3.3V? Proveriti da li to MCU vec radi!"
- note added: "USB-C Connector"
- note removed: "Buck-Boost Converter"
- title: Battery Managment System (DAC) -> Battery Managment System (BMS)
- moved on the sheet: BAT, C1, C10, C2, C3, C4, C5, C6, C7, C8, C9, L1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

Commit message: *
Parts:
- added D1: D_Small, symbol Device:D_Small
- added R19, R20, R21, R22: 0, symbol Device:R_Small
- added U6: USBLC6-2SC6, fpl:USBLC6-2SC6, symbol syl:USBLC6-2SC6
- BAT1: renamed from BAT; footprint (none) -> Battery:BatteryHolder_MPD_BH-18650-PC2
- USB1: LCSC Part C309365 -> (none); LCSCPart (none) -> C309365
- renumbered C2 to C1, C4 to C10, C5 to C2, C6 to C3, C7 to C4, C1 to C5, C8 to C6, C9 to C7, C10 to C8, C3 to C9, R6 to R10, R10 to R11, R7 to R12, R8 to R13, R4 to R14, R14 to R2, R2 to R3, R3 to R4, R12 to R5, R13 to R6, R11 to R7, R5 to R8, U3 to U1, U4 to U3, U1 to U4
Connections:
- net +USB_D: now also U6.3, U6.6
- net -USB_D: now also U6.1, U6.4
- net BATSYS: now also R20.1, R20.2
- net BCKOUT5: now also R21.2; no longer C4.2, C6.2, U1.1 (VOUT), U1.10 (FB)
- net BCOUT: now also R22.1, R22.2
- net GND: now also U6.2
- net VBUS: now also D1.1 (K), D1.2 (A), R19.1, U6.5; no longer U2.13 (IN)
- new net BCK5_VOUT: C4.2, C6.2, R21.1, U1.1 (VOUT), U1.10 (FB)
- new net VBSIN: R19.2, U2.13 (IN)
Other:
- note removed: "Povuci D+ na 3.3V? Proveriti da li to MCU vec radi!"
- moved on the sheet: C7, C8, L2, U3
