File: device/hw/$pr/Sheets/South Bridge/bms.kicad_sch (KiCad schematic)
At the start: 47 parts, among them U1 TPS63002DRCT, U2 BQ24074RGTR, U3 TPS62082DSGR, U4 BQ27441DRZR-G1B, U6 USBLC6-2SC6, U7 TS3USB221ARSER

Commit message: application
Parts:
- removed D1: D_Small, symbol Device:D_Small
- removed R10, R8, R9: 5.1k, symbol Device:R
- removed R5, R6: 100k, symbol Device:R
- added R11: 10k, symbol Device:R
- added R13: 0, symbol Device:R_Small
- added R32, R33, R34: 5.1k, symbol Device:R_Small
- added R5, R6: 100k, symbol Device:R_Small
- added SW3: SW_SPDT, symbol Switch:SW_SPDT
Connections:
- net BCKOUT33: now also R32.2, R33.2, R34.2, R5.1, R6.1, SW3.3 (C)
- net CHG_CHG: now also R5.2
- net CHG_PGOOD: now also R6.2
- net FG_GPOUT: now also R32.1
- net GND: now also SW3.1 (A); no longer D3.1 (K)
- net IICGAUG_SCL: now also R34.1
- net IICGAUG_SDA: now also R33.1
- net USB_SLC: now also R13.2
- net BCK5_EN: now reaches C3.2, R2.1, U1.6 (EN), U1.7 (PS/SYNC), U1.8 (VINA)
- new net: R11.2, R13.1
- new net: R11.1, SW3.2 (B)
- new net GNDLD: D3.1 (K)
Other:
- note added: "1."
- note added: "Birač za USB Input Source"
- note added: "USB-C Konektor, [USBLC6-2SC6] TVS Diode Protection i [TS3USB221ARSER] 1:2 Multiplexer za USB Host"
- note added: "[BQ24074RGTR] IC za punjenje i pražnjenje baterije. 1. NTC Thermistor (Promenljivi otpornik) za praćenje temperature baterije."
- note added: "[BQ27441DRZR-G1B] IC za praćenje stanja baterije i [BAT1 (SAMSUNG20R)] 2000mAh baterija."
- note added: "[TPS62082DSGR] Fiksni 3.3V Step-Down konverter BCKOUT5(TPS63002DRCT)-->BCKOUT33(TPS62082DSGR)"
- note added: "[TPS63002DRCT] Fiksni 5V Boost konverter BCOUT(BQ24074RGTR)-->BCKOUT5(TPS63002DRCT)"
- note removed: "!Mora biti blizu BAT!"
- moved on the sheet: BAT1, C1, C10, C2, C28, C3, C4, C5, C6, C7, C8, C9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

Commit message: application
Parts:
- removed D3, D4: LED, symbol Device:LED
- removed R19, R20, R21, R22: 0, symbol Device:R_Small
- removed R24, R27: 220, symbol Device:R_Small
- removed R26: 10k, symbol Device:R_Small
- added D1, D10: LED, LED_SMD:LED_0805_2012Metric, symbol Device:LED
- added D2, D5, D6: LED, LED_SMD:LED_0603_1608Metric, symbol Device:LED
- added Q4, Q5: NPN, Package_TO_SOT_SMD:SOT-23, symbol Simulation_SPICE:NPN
- added R2: 0, symbol Device:R_Small
- added R35, R37: 4.7k, symbol Device:R_Small
- BAT1: footprint Battery:BatteryHolder_MPD_BH-18650-PC2 -> fpl:BAT-TH_BH-18650-A5BJ003; LCSCPart (none) -> C5371778
- C1: renamed from C28; footprint (none) -> Capacitor_SMD:C_0603_1608Metric; LCSCPart (none) -> C14663
- C10: renamed from C9; footprint (none) -> Capacitor_SMD:C_0603_1608Metric; LCSCPart (none) -> C15849
- C11: renamed from C10; footprint (none) -> Capacitor_SMD:C_0603_1608Metric; LCSCPart (none) -> C15849
- C2: renamed from C5; footprint (none) -> Capacitor_SMD:C_0805_2012Metric; LCSCPart (none) -> C1779
- C3: renamed from C1; footprint (none) -> Capacitor_SMD:C_0603_1608Metric; LCSCPart (none) -> C15849
- C4: renamed from C2; footprint (none) -> Capacitor_SMD:C_0805_2012Metric; LCSCPart (none) -> C15850
- C5: renamed from C4; footprint (none) -> Capacitor_SMD:C_0805_2012Metric; LCSCPart (none) -> C15850
- C6: footprint (none) -> Capacitor_SMD:C_0805_2012Metric; LCSCPart (none) -> C15850
- C7: renamed from C3; footprint (none) -> Capacitor_SMD:C_0603_1608Metric; LCSCPart (none) -> C14663
- C8: renamed from C7; footprint (none) -> Capacitor_SMD:C_0805_2012Metric; LCSCPart (none) -> C15850
- C9: renamed from C8; footprint (none) -> Capacitor_SMD:C_0805_2012Metric; LCSCPart (none) -> C45783
- L1: footprint (none) -> Inductor_SMD:L_1008_2520Metric; LCSCPart (none) -> C3002551
- L2: footprint (none) -> Capacitor_SMD:C_0603_1608Metric; LCSCPart (none) -> C15849
- R10: renamed from R15; footprint (none) -> Resistor_SMD:R_0402_1005Metric; LCSCPart (none) -> C25905
- R11: renamed from R3; footprint (none) -> Resistor_SMD:R_0603_1608Metric; LCSCPart (none) -> C13167
- R12: renamed from R16; footprint (none) -> Resistor_SMD:R_0402_1005Metric; LCSCPart (none) -> C25905
- R13: renamed from R1; footprint (none) -> Resistor_SMD:R_0603_1608Metric; LCSCPart (none) -> C23253
- R14: renamed from R5; footprint (none) -> Resistor_SMD:R_0603_1608Metric; LCSCPart (none) -> C25803
- R15: renamed from R6; footprint (none) -> Resistor_SMD:R_0603_1608Metric; LCSCPart (none) -> C25803
- R17: renamed from R11; footprint (none) -> Resistor_SMD:R_0402_1005Metric; LCSCPart (none) -> C25744
- R18: renamed from R13; footprint (none) -> Resistor_SMD:R_0805_2012Metric; LCSCPart (none) -> C17477
- R19: renamed from R34; footprint (none) -> Resistor_SMD:R_0402_1005Metric; LCSCPart (none) -> C25905
- R20: renamed from R33; footprint (none) -> Resistor_SMD:R_0402_1005Metric; LCSCPart (none) -> C25905
- R21: renamed from R32; footprint (none) -> Resistor_SMD:R_0402_1005Metric; LCSCPart (none) -> C25905
- R22: renamed from R14; footprint (none) -> Resistor_SMD:R_1206_3216Metric; LCSCPart (none) -> C601085
- R24: renamed from R12; footprint (none) -> Resistor_SMD:R_0402_1005Metric; LCSCPart (none) -> C25744
- R4: footprint (none) -> Resistor_SMD:R_0603_1608Metric; LCSCPart (none) -> C22765
- R7: footprint (none) -> Resistor_SMD:R_0402_1005Metric; LCSCPart (none) -> C25744
- R8: renamed from R25; footprint (none) -> Resistor_SMD:R_0402_1005Metric; LCSCPart (none) -> C25744
- R9: renamed from R2; footprint (none) -> Resistor_SMD:R_0603_1608Metric; LCSCPart (none) -> C22775
- U1: renamed from U7; LCSCPart (none) -> C128396
- renumbered SW3 to SW1, U1 to U3, U6 to U4, U3 to U5, U4 to U6
Connections:
- net BCK5_VOUT is gone; now on net BCKOUT5: C5.2, C6.2, U3.1 (VOUT), U3.10 (FB)
- net VBSIN is gone; now on net VBUS: U2.13 (IN)
- net BCKOUT33: now also D2.2 (A), R35.1, R37.1
- net BCKOUT5: now also Q4.3 (E), R2.2
- net USB_SLC: now also U1.9 (S)
- net VBUS: now also Q5.2 (B), Q5.3 (E)
- net at R17.1, SW1.2 (B): now also D5.2 (A), D6.1 (K)
- new net: D10.2 (A), Q5.1 (C), R37.2
- new net: D1.2 (A), Q4.1 (C), R35.2
- new net: Q4.2 (B), R2.1
- new net LGND: D1.1 (K), D10.1 (K), D2.1 (K), D5.1 (K)
- new net LVCC: D6.2 (A)
Other:
- note added: "Logic Level Shifter za LED"
- note added: "[BQ24074RGTR] IC za punjenje i pražnjenje baterije."
- note removed: "1."
- note removed: "[BQ24074RGTR] IC za punjenje i pražnjenje baterije. 1. NTC Thermistor (Promenljivi otpornik) za praćenje temperature baterije."
- moved on the sheet: BAT1, C10, C11, C2, C3, C4, C5, C6, C7, C8, C9, L1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

Commit message: application
Parts:
- removed D1, D10: LED, LED_SMD:LED_0805_2012Metric, symbol Device:LED
- removed Q4, Q5: NPN, Package_TO_SOT_SMD:SOT-23, symbol Simulation_SPICE:NPN
- removed R2: 0, symbol Device:R_Small
- removed R35, R37: 4.7k, symbol Device:R_Small
- added D3, D5: LED, LED_SMD:LED_0603_1608Metric, symbol Device:LED
- added R12, R24: 220, symbol Device:R_Small
- added R23, R6, R7: 47, symbol Device:R_Small
- added R8, R9: 0, Resistor_SMD:R_0805_2012Metric, symbol Device:R_Small
- renumbered C5 to C10, C6 to C11, C3 to C2, C10 to C3, C11 to C4, C2 to C5, C8 to C6, C4 to C7, C7 to C8, D5 to D1, D6 to D2, D2 to D4, R10 to R1, R19 to R10, R20 to R11, R24 to R13, R21 to R14, R13 to R15, R11 to R16, R4 to R17, R22 to R18, R7 to R19, R12 to R2, R14 to R20, R15 to R21, R9 to R22, R8 to R3, R17 to R4, R18 to R5, U4 to U1, U1 to U2, U6 to U3, U2 to U4, U3 to U6
Connections:
- net BCKOUT5: now also D5.2 (A)
- net GND: now also R12.1, R24.1
- net LGND: now also R23.1, R8.2; no longer D1.1 (K), D4.1 (K)
- net LVCC: now also R9.2; no longer D2.2 (A)
- net VBUS: now also D3.2 (A)
- new net: D2.2 (A), R7.1
- new net: R7.2, R9.1
- new net: D1.1 (K), R6.1
- new net: R6.2, R8.1
- new net: D3.1 (K), R12.2
- new net: D5.1 (K), R24.2
- new net: D4.1 (K), R23.2
Other:
- note added: "Buck-Boost Fixed 3.3 Converter"
- note removed: "Buck-StepDown Fixed 3.3 Converter"
- note removed: "Logic Level Shifter za LED"
- moved on the sheet: BAT1, C10, C11, C2, C3, C4, C5, C7, C8, D1, D2, L1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
