File: device/hw/$pr/Sheets/South Bridge/stm32_mcu.kicad_sch (KiCad schematic)
At the start: 0 parts

Commit message: BMS
Other:
- company: (none) -> ETŠ Mihajlo Pupin "Medmentum"
Changed lines of the file:
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@@
 	(generator_version "8.0")
 	(paper "A4")
+	(title_block
+		(company "ETŠ Mihajlo Pupin \"Medmentum\"")
+	)
 )

Commit message: application
Parts:
- added U5: STM32F411CEU6, fpl:STM32F411CEU6, symbol syl:STM32F411CEU6
Connections:
- new net: U5.23 (VSS), U5.35 (VSS), U5.47 (VSS), U5.49 (VSS)
- new net: U5.24 (VDD), U5.36 (VDD), U5.48 (VDD)
Changed lines of the file:
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@@
 		(company "ETŠ Mihajlo Pupin \"Medmentum\"")
 	)
+	(symbol
+		(lib_id "syl:STM32F411CEU6")
+		(at 140.97 88.9 0)
+		(unit 1)
+		(exclude_from_sim no)
+		(in_bom yes)
+		(on_board yes)
+		(dnp no)
+		(fields_autoplaced yes)
+		(property "Reference" "U5"
+			(at 140.97 38.1 0)
+			(effects
+				(font
+					(size 1.27 1.27)
+				)
+			)
+		)
+		(property "Value" "STM32F411CEU6"
+			(at 140.97 40.64 0)
+			(effects
+				(font
+					(size 1.27 1.27)
+				)
+			)
+		)
+		(property "Footprint" "fpl:STM32F411CEU6"
+			(at 140.97 88.9 0)
+			(effects
+				(font
+					(size 1.27 1.27)
+				)
+				(justify bottom)
+				(hide yes)
+			)
+		)
+		(property "Datasheet" "https://github.com/nskemish/medmentum/blob/main/device/hw/%24ds/South%20Bridge/STM32/STM32F411CEU6.pdf"
+			(at 140.97 88.9 0)
+			(effects
+				(font
+					(size 1.27 1.27)
+				)
+				(hide yes)
+			)
+		)
+		(property "Description" ""
+			(at 140.97 88.9 0)
+			(effects
+				(font
+					(size 1.27 1.27)
+				)
+				(hide yes)
+			)
+		)
+		(property "Package" "UFQFPN-48"
+			(at 140.97 88.9 0)
+			(effects
+				(font
+					(size 1.27 1.27)
+				)
+				(justify bottom)
+				(hide yes)
+			)
+		)
+		(property "MP" "STM32F411CEU6"
+			(at 140.97 88.9 0)
+			(effects
+				(font
+					(size 1.27 1.27)
+				)
+				(justify bottom)
+				(hide yes)
+			)
+		)
+		(property "LCSCPart" "C60420"
+			(at 140.97 43.18 0)
+			(effects
+				(font
+					(size 1.27 1.27)
+				)
+			)
+		)
+		(pin "17"
+		)
+		(pin "34"
+		)
+		(pin "27"
+		)
+		(pin "3"
+		)
+		(pin "22"
+		)
+		(pin "18"
+		)
+		(pin "45"
+		)
+		(pin "37"
+		)
+		(pin "4"
+		)
+		(pin "43"
+		)
+		(pin "6"
+		)
+		(pin "9"
+		)
+		(pin "2"
+		)
+		(pin "29"
+		)
+		(pin "41"
+		)
+		(pin "31"
+		)
+		(pin "32"
+		)
+		(pin "42"
+		)
+		(pin "23"
+		)
+		(pin "38"
+		)
+		(pin "36"
+		)
+		(pin "20"
+		)
+		(pin "8"
+		)
+		(pin "48"
+		)
+		(pin "5"
+		)
+		(pin "28"
+		)
+		(pin "30"
+		)
+		(pin "19"
+		)
+		(pin "16"
+		)
+		(pin "44"
+		)
+		(pin "33"
+		)
+		(pin "40"
+		)
+		(pin "49"
+		)
+		(pin "46"
+		)
+		(pin "47"
+		)
+		(pin "11"
+		)
+		(pin "35"
+		)
+		(pin "25"
+		)
+		(pin "14"
+		)
+		(pin "13"
+		)
+		(pin "7"
+		)
+		(pin "39"
+		)
+		(pin "21"
+		)
+		(pin "12"
+		)
+		(pin "26"
+		)
+		(pin "15"
+		)
+		(pin "24"
+		)
+		(pin "1"
+		)
+		(pin "10"
+		)
+		(instances
+			(project ""
+				(path "/ead52261-b3da-41ef-908f-3daaabe10954/940ef1bd-73e9-475b-b1ba-056ab9b45d18/e562aa6d-779d-4ead-8af2-051e7c1e0296"
+					(reference "U5")
+					(unit 1)
+				)
+			)
+		)
+	)
 )

Commit message: *
Parts:
- added C11, C18, C22, C26: 4.7u, symbol Device:C
- added C12, C13, C14, C15, C16, C17, C21, C25: 100n, symbol Device:C
- added C19, C20: 16p, symbol Device:C
- added C23, C24: 5p, symbol Device:C
- added FB1: 100R@100MHz, Inductor_SMD:L_0805_2012Metric, symbol Device:FerriteBead
- added R17: 100k, symbol Device:R
- added R18: 10k, symbol Device:R
- added SW1: SW_Push, symbol Switch:SW_Push
- added SW2: SW_SPDT, symbol Switch:SW_SPDT
- added Y1: 18pF, Crystal:Crystal_SMD_3225-4Pin_3.2x2.5mm, symbol Device:Crystal_GND24_Small
- added Y2: 12.5pF, Crystal:Crystal_SMD_3215-2Pin_3.2x1.5mm, symbol Device:Crystal_Small
Connections:
- net BCKOUT33: now reaches U5.1 (VBAT)
- net BCKOUT33: now also U5.24 (VDD), U5.36 (VDD), U5.48 (VDD), C11.2, C12.2, C13.2, C14.2, C15.2, C16.2, C17.2, C26.2, FB1.1, R17.1, SW2.3 (C)
- net at U5.22 (VCAP_1): now also C22.2
- net GNDD: now reaches U5.23 (VSS), U5.35 (VSS), U5.47 (VSS), U5.49 (VSS)
- net GNDD: now also C11.1, C12.1, C13.1, C14.1, C15.1, C16.1, C17.1, C19.2, C20.1, C22.1, C23.2, C24.1, C25.1, SW1.1, SW2.1 (A), Y1.2, Y1.4
- net LSE_IN: now reaches U5.3 (PC14-OSC32_IN)
- net LSE_IN: now also C23.1, Y2.2
- net LSE_OUT: now reaches U5.4 (PC15-OSC32_OUT)
- net LSE_OUT: now also C24.2, Y2.1
- net BOOT0: now reaches U5.44 (BOOT0)
- net BOOT0: now also R18.2
- net HSE_IN: now reaches U5.5 (PH0-OSC_IN)
- net HSE_IN: now also C19.1, Y1.1
- net HSE_OUT: now reaches U5.6 (PH1-OSC_OUT)
- net HSE_OUT: now also C20.2, Y1.3
- net NRST: now reaches U5.7 (NRST)
- net NRST: now also C25.2, R17.2, SW1.2
- net GNDA: now reaches U5.8 (VSSA)
- net GNDA: now also C18.1, C21.1, C26.1
- net VDDA: now reaches U5.9 (VREF+)
- net VDDA: now also C18.2, C21.2, FB1.2
- new net SW_BOOT0: R18.1, SW2.2 (B)
