File: device/hw/$pr/Sheets/South Bridge/stm32_mcu.kicad_sch (KiCad schematic)
At the start: 26 parts, among them SW1 SW_Push, SW2 SW_SPDT, U5 STM32F411CEU6, Y1 18pF, Y2 12.5pF

Commit message: application
Parts:
- added R31: 0, symbol Device:R_Small
Connections:
- net BCKOUT33: now also R31.1; no longer C11.2, C12.2, C13.2, C14.2, C15.2, C16.2, C17.2, U5.1 (VBAT), U5.24 (VDD), U5.36 (VDD), U5.48 (VDD)
- net LEDPWM renamed LEDHOPWM
- net VDDA renamed VDDASTM
- new net VDD: C11.2, C12.2, C13.2, C14.2, C15.2, C16.2, C17.2, R31.2, U5.1 (VBAT), U5.24 (VDD), U5.36 (VDD), U5.48 (VDD)
Changed lines of the file:
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@@
-	(wire
-		(pts
-			(xy 81.28 53.34) (xy 86.36 53.34)
-		)
-		(stroke
-			(width 0)
-			(type default)
-		)
-	)
 	(wire
 		(pts
@@
 		(pts
 			(xy 121.92 109.22) (xy 124.46 106.68)
+		)
+		(stroke
+			(width 0)
+			(type default)
+		)
+	)
+	(wire
+		(pts
+			(xy 85.09 53.34) (xy 86.36 53.34)
 		)
 		(stroke
@@
 	(text "TIM2"
 		(exclude_from_sim no)
-		(at 175.006 120.904 0)
+		(at 176.276 120.904 0)
 		(effects
 			(font
@@
 		)
 	)
-	(label "VDD"
+	(label "VDDSTM"
 		(at 127 53.34 0)
 		(fields_autoplaced yes)
@@
 		)
 	)
-	(label "VDDA"
+	(label "VDDASTM"
 		(at 124.46 67.31 0)
 		(fields_autoplaced yes)
@@
 		)
 	)
-	(hierarchical_label "LEDPWM"
+	(hierarchical_label "LEDHOPWM"
 		(shape input)
 		(at 168.91 120.65 0)
@@
 	)
 	(symbol
+		(lib_id "Device:R_Small")
+		(at 82.55 53.34 90)
+		(unit 1)
+		(exclude_from_sim no)
+		(in_bom yes)
+		(on_board yes)
+		(dnp no)
+		(property "Reference" "R31"
+			(at 82.55 50.292 90)
+			(effects
+				(font
+					(size 0.635 0.635)
+				)
+			)
+		)
+		(property "Value" "0"
+			(at 82.55 51.562 90)
+			(effects
+				(font
+					(size 0.635 0.635)
+				)
+			)
+		)
+		(property "Footprint" ""
+			(at 82.55 53.34 0)
+			(effects
+				(font
+					(size 1.27 1.27)
+				)
+				(hide yes)
+			)
+		)
+		(property "Datasheet" "~"
+			(at 82.55 53.34 0)
+			(effects
+				(font
+					(size 1.27 1.27)
+				)
+				(hide yes)
+			)
+		)
+		(property "Description" "Resistor, small symbol"
+			(at 82.55 53.34 0)
+			(effects
+				(font
+					(size 1.27 1.27)
+				)
+				(hide yes)
+			)
+		)
+		(pin "1"
+		)
+		(pin "2"
+		)
+		(instances
+			(project "medmentum"
+				(path "/ead52261-b3da-41ef-908f-3daaabe10954/940ef1bd-73e9-475b-b1ba-056ab9b45d18/e562aa6d-779d-4ead-8af2-051e7c1e0296"
+					(reference "R31")
+					(unit 1)
+				)
+			)
+		)
+	)
+	(symbol
 		(lib_id "power:GNDD")
 		(at 127 104.14 90)
@@
 	(symbol
 		(lib_id "power:+BATT")
-		(at 81.28 53.34 90)
+		(at 80.01 53.34 90)
 		(unit 1)
 		(exclude_from_sim no)
@@
 		(on_board yes)
 		(dnp no)
-		(fields_autoplaced yes)
 		(property "Reference" "#PWR037"
-			(at 85.09 53.34 0)
+			(at 83.82 53.34 0)
 			(effects
 				(font
@@
 		)
 		(property "Value" "BCKOUT33"
-			(at 77.47 53.34 90)
+			(at 76.2 53.34 90)
 			(effects
 				(font
@@
 		)
 		(property "Footprint" ""
-			(at 81.28 53.34 0)
+			(at 80.01 53.34 0)
 			(effects
 				(font
@@
 		)
 		(property "Datasheet" ""
-			(at 81.28 53.34 0)
+			(at 80.01 53.34 0)
 			(effects
 				(font
@@
 		)
 		(property "Description" "Power symbol creates a global label with name \"+BATT\""
-			(at 81.28 53.34 0)
-			(effects
-				(font
+			(at 80.01 53.34 0)
+			(effects
+				(font

Commit message: application
Parts:
- added D8, D9: D_Small, Diode_SMD:D_SOD-323, symbol Device:D_Small
- added Q2, Q3: NPN, Package_TO_SOT_SMD:SOT-23, symbol Simulation_SPICE:NPN
- added R1, R3, R38, R39, R40: R, symbol Device:R_Small
- C12: renamed from C11; footprint (none) -> Capacitor_SMD:C_0805_2012Metric; LCSCPart (none) -> C1779
- C13: renamed from C12; footprint (none) -> Capacitor_SMD:C_0603_1608Metric; LCSCPart (none) -> C14663
- C14: renamed from C13; footprint (none) -> Capacitor_SMD:C_0603_1608Metric; LCSCPart (none) -> C14663
- C15: renamed from C14; footprint (none) -> Capacitor_SMD:C_0603_1608Metric; LCSCPart (none) -> C14663
- C16: renamed from C15; footprint (none) -> Capacitor_SMD:C_0603_1608Metric; LCSCPart (none) -> C14663
- C17: renamed from C16; footprint (none) -> Capacitor_SMD:C_0603_1608Metric; LCSCPart (none) -> C14663
- C18: renamed from C17; footprint (none) -> Capacitor_SMD:C_0603_1608Metric; LCSCPart (none) -> C14663
- C19: renamed from C26; footprint (none) -> Capacitor_SMD:C_0805_2012Metric; LCSCPart (none) -> C1779
- C20: renamed from C18; footprint (none) -> Capacitor_SMD:C_0805_2012Metric; LCSCPart (none) -> C1779
- C21: footprint (none) -> Capacitor_SMD:C_0603_1608Metric; LCSCPart (none) -> C14663
- C22: renamed from C23; footprint (none) -> Capacitor_SMD:C_0402_1005Metric; LCSCPart (none) -> C880630
- C23: renamed from C24; footprint (none) -> Capacitor_SMD:C_0402_1005Metric; LCSCPart (none) -> C880630
- C24: renamed from C19; footprint (none) -> Capacitor_SMD:C_0402_1005Metric; LCSCPart (none) -> C48836
- C25: renamed from C20; footprint (none) -> Capacitor_SMD:C_0402_1005Metric; LCSCPart (none) -> C48836
- C26: renamed from C25; footprint (none) -> Capacitor_SMD:C_0603_1608Metric; LCSCPart (none) -> C14663
- C27: renamed from C22; footprint (none) -> Capacitor_SMD:C_0805_2012Metric; LCSCPart (none) -> C1779
- D3: renamed from D2; footprint (none) -> LED_SMD:LED_0603_1608Metric; LCSCPart (none) -> C2290
- R23: value 220 -> R
- R25: renamed from R31; footprint (none) -> Resistor_SMD:R_0805_2012Metric; LCSCPart (none) -> C17477
- R27: renamed from R18; footprint (none) -> Resistor_SMD:R_0402_1005Metric; LCSCPart (none) -> C25744
- R28: renamed from R17; footprint (none) -> Resistor_SMD:R_0603_1608Metric; LCSCPart (none) -> C25803
- renumbered SW1 to SW3, U5 to U7, Y2 to Y1, Y1 to Y2
Connections:
- net BCKOUT33: now also R40.2
- net FG_GPOUT: now also U7.26 (PB13); no longer U7.29 (PA8)
- net GNDD: now also Q2.3 (E), Q3.3 (E); no longer D3.1 (K)
- net LEDHOPWM: now also R1.2; no longer U7.14 (PA4)
- net SW_BOOT0: now also D3.2 (A); no longer R23.2
- net PANICPWM1: now reaches U7.11 (PA1)
- net at U7.12 (PA2): now also R3.2
- net at U7.13 (PA3): now also R1.1
- net PANICGPIO: now reaches U7.25 (PB12)
- net DISPEN: now reaches U7.34 (PA13)
- net LEDEN: now reaches U7.37 (PA14)
- net LEDEN: now also D8.2 (A)
- net CONFSW: now reaches U7.41 (PB5)
- net HOSW: now reaches U7.45 (PB8)
- net at R23.1: now also Q2.1 (C); no longer D3.2 (A)
- new net: D8.1 (K), D9.1 (K), R38.1
- new net: Q3.2 (B), R38.2
- new net: Q2.2 (B), R39.2
- new net BUZPWM: U7.29 (PA8)
- new net DBSW: D9.2 (A)
- new net LEDCHPWM: R3.1
- new net LGND: D3.1 (K), R23.2
- new net LVCC: Q3.1 (C), R39.1, R40.1
Other:
- note added: "TIM1"
- moved on the sheet: D3

Commit message: application
Parts:
- removed D3: LED, LED_SMD:LED_0603_1608Metric, symbol Device:LED
- removed D8, D9: D_Small, Diode_SMD:D_SOD-323, symbol Device:D_Small
- removed Q3: NPN, Package_TO_SOT_SMD:SOT-23, symbol Simulation_SPICE:NPN
- removed R23: R, symbol Device:R_Small
- removed R28: 100k, Resistor_SMD:R_0603_1608Metric, symbol Device:R
- added D6, D7: LED, LED_SMD:LED_0603_1608Metric, symbol Device:LED
- added Q1: PNP, symbol Simulation_SPICE:PNP
- added R26, R30: 0, symbol Device:R_Small
- added R27, R28, R34, R35: 47, symbol Device:R_Small
- added R32, R33, R37: 5.1k, Resistor_SMD:R_0402_1005Metric, symbol Device:R_Small
- R31: renamed from R1; value R -> 47
- R36: renamed from R3; value R -> 47
- R38: value R -> 5.1k; footprint (none) -> Resistor_SMD:R_0402_1005Metric; LCSCPart (none) -> C25905
- R39, R40: value R -> 1k
- renumbered C19 to C16, C16 to C17, C17 to C18, C22 to C19, C23 to C20, C24 to C21, C25 to C22, C26 to C23, C20 to C24, C18 to C25, C27 to C26, C21 to C27, R27 to R29
Connections:
- net BCKOUT33: now also Q1.3 (E); no longer R40.2
- net GNDD: now also R38.1, R32.2, R33.1, R37.1
- net IICDISP_SCL: now also R33.2
- net IICDISP_SDA: now also R32.1
- net IICGAUG_SCL: now also R37.2
- net IICGAUG_SDA: now also R38.2
- net LGND: now also Q2.1 (C), R30.1
- net LVCC: now also Q1.1 (C), R26.2; no longer R39.1
- net SW_BOOT0: now also D6.1 (K), D7.2 (A)
- net UARTRX_ESP: now also R34.2; no longer U7.31 (PA10)
- net UARTTX_ESP: now also R35.2; no longer U7.30 (PA9)
- net at Q2.2 (B): now also R40.2; no longer R39.2
- net LEDEN: no longer names the net of U7.37 (PA14)
- net LEDEN: now also R39.1
- new net: R26.1, R27.2
- new net: R28.1, R30.2
- new net: Q1.2 (B), R39.2
- new net: D6.2 (A), R27.1
- new net: D7.1 (K), R28.2
- new net STM_UARTRX: R34.1, U7.31 (PA10)
- new net STM_UARTTX: R35.1, U7.30 (PA9)
Other:
- note added: "1."
- note added: "2."
- note added: "3."
- note added: "4."
- note added: "5."
- note added: "6."
- note added: "7."
- note added: "8."
- note added: "Boot memory picker."
- note added: "HSE (High Speed External) Clock."
- note added: "IIC "Pull-up" otpornici."
- note added: "LED Debug mode picker."
- note added: "LSE (Low Speed External) Clock."
- note added: "Reset."
- note added: "STM32F411CE MCU"
- note added: "Čišćenje signala od šuma za analogno napajanje."
- note added: "Čišćenje signala od šuma za digitalno napajanje."
- moved on the sheet: C12, C13, C14, C15, C16, C17, C18, C19, C20, C21, C22, C23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
