File: device/hw/$pr/Sheets/South Bridge/stm32_mcu.kicad_sch (KiCad schematic)
At the start: 115 parts, among them CON2 ZX-IDC2.54-2-13PZZ, Q1 PNP, Q2 NPN, Q4 NPN, SW2 SW_SPDT, SW3 SW_Push, SW6 SW_SPDT, SW7 SW_Push, SW8 SW_SPDT, U10 BQ24074RGTR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

Commit message: application
Connections:
- net CHG_CHG renamed CHG_#CHG
- net CHG_PGOOD renamed CHG_#PGOOD
- net IICGAUG_SCL renamed FG_SCL
- net IICGAUG_SDA renamed FG_SDA
Other:
- note added: "Buck-Boost Fixed 3.3V Converter"
- note removed: "Buck-Boost Fixed 3.3 Converter"
- moved on the sheet: BAT2, C44, C45, R67, R68, R69, R70, R71, U14
