File: device/hw/$pr/Sheets/North Bridge/esp32_mcu.kicad_sch (KiCad schematic)
At the start: 0 parts

Commit message: BMS
Other:
- company: (none) -> ETŠ Mihajlo Pupin "Medmentum"
Changed lines of the file:
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@@
 	(generator_version "8.0")
 	(paper "A4")
+	(title_block
+		(company "ETŠ Mihajlo Pupin \"Medmentum\"")
+	)
 )

Commit message: application
Parts:
- added C27: 4.7u, symbol Device:C
- added C29, C31, C32: 100n, symbol Device:C
- added C30: 1u, symbol Device:C
- added R30: 10k, symbol Device:R
- added U8: ESP32-C3-MINI-1-H4, fpl:ESP32-C3-MINI-1-H4, symbol syl:ESP32-C3-MINI-1-H4(4MB)
Connections:
- new net: U8.10 (NC), U8.15 (NC), U8.17 (NC), U8.24 (NC), U8.25 (NC), U8.28 (NC), U8.29 (NC), U8.32 (NC), U8.33 (NC), U8.34 (NC), U8.35 (NC), U8.4 (NC), U8.7 (NC), U8.9 (NC)
- new net: C30.2, R30.1, U8.8 (EN)
- new net +USB_DESP: U8.27 (IO19)
- new net -USB_DESP: U8.26 (IO18)
- new net BCKOUT33: C27.2, C29.2, C31.2, C32.2, R30.2, U8.3 (3V3)
- new net GNDD: C27.1, C29.1, C30.1, C31.1, C32.1, U8.1 (GND), U8.11 (GND), U8.14 (GND), U8.2 (GND), U8.36 (GND), U8.37 (GND), U8.38 (GND), U8.39 (GND), U8.40 (GND), U8.41 (GND), U8.42 (GND), U8.43 (GND), U8.44 (GND), U8.45 (GND), U8.46 (GND), U8.47 (GND), U8.48 (GND), U8.49 (GND), U8.50 (GND), U8.51 (GND), U8.52 (GND), U8.53 (GND)
- new net UARTRX_ESP: U8.31 (TXD0)
- new net UARTTX_ESP: U8.30 (RXD0)
- no-connect marks 0 -> 12

Commit message: application
Connections:
- net ENESP: now reaches C30.2, R30.1, U8.8 (EN)
Changed lines of the file:
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@@
+		)
+	)
+	(label "ENESP"
+		(at 134.62 64.77 0)
+		(fields_autoplaced yes)
+		(effects
+			(font
+				(size 0.508 0.508)
+			)
+			(justify left bottom)
+		)
+	)
+	(label "VDDESP"
+		(at 134.62 55.88 0)
+		(fields_autoplaced yes)
+		(effects
+			(font
+				(size 0.508 0.508)
+			)
+			(justify left bottom)
 		)
 	)

Commit message: application
Parts:
- added C32: 100n, Capacitor_SMD:C_0603_1608Metric, symbol Device:C
- added D4: LED, LED_SMD:LED_0603_1608Metric, symbol Device:LED
- added R30, R32: 10k, Resistor_SMD:R_0402_1005Metric, symbol Device:R_Small
- added SW4: SW_Push, symbol Switch:SW_Push
- added SW5: SW_SPDT, symbol Switch:SW_SPDT
- C28: renamed from C27; footprint (none) -> Capacitor_SMD:C_0805_2012Metric; LCSCPart (none) -> C1779
- C29: renamed from C32; footprint (none) -> Capacitor_SMD:C_0603_1608Metric; LCSCPart (none) -> C14663
- C30: renamed from C31; footprint (none) -> Capacitor_SMD:C_0603_1608Metric; LCSCPart (none) -> C14663
- C31: renamed from C29; footprint (none) -> Capacitor_SMD:C_0603_1608Metric; LCSCPart (none) -> C14663
- C33: renamed from C30; footprint (none) -> Capacitor_SMD:C_0603_1608Metric; LCSCPart (none) -> C15849
- R29: renamed from R30; footprint (none) -> Resistor_SMD:R_0402_1005Metric; LCSCPart (none) -> C25744
Connections:
- net BCKOUT33: now also R30.1, R32.2, SW5.1 (A)
- net ENESP: now also C32.1, SW4.1
- net GNDD: now also C32.2, D4.1 (K), SW4.2, SW5.3 (C)
- net at U8.22 (IO8): now also R32.1
- net at U8.23 (IO9): now also D4.2 (A), SW5.2 (B)
- net at U8.5 (IO2): now also R30.2
- no-connect marks 12 -> 9
Other:
- note added: "GPIO9 SPI 1 GPIO9 Joint Download Boot USB 0"
- moved on the sheet: C28, C29, C30, C31, C33, R29, U8

Commit message: application
Parts:
- removed D4: LED, LED_SMD:LED_0603_1608Metric, symbol Device:LED
- added C34: 1u, Capacitor_SMD:C_0603_1608Metric, symbol Device:C
- added D8, D9: LED, LED_SMD:LED_0603_1608Metric, symbol Device:LED
- added R44: 10k, Resistor_SMD:R_0402_1005Metric, symbol Device:R
- added R45, R46: 47, symbol Device:R_Small
- renumbered C32 to C28, C28 to C29, C29 to C30, C30 to C31, C33 to C32, C31 to C33, R30 to R41, R29 to R42, R32 to R43
Connections:
- net BCKOUT33: now also C29.1, C30.1, C31.1, C33.1, SW5.3 (C); no longer C29.2, C30.2, C31.2, C33.2, SW5.1 (A)
- net GNDD: now also C29.2, C30.2, C31.2, C32.2, C33.2, SW5.1 (A), C34.1; no longer C29.1, C30.1, C31.1, C32.1, C33.1, SW5.3 (C)
- net at U8.23 (IO9): now also R44.2; no longer SW5.2 (B)
- net at R41.2, U8.5 (IO2): now also C34.2
- net ENESP renamed ENRST
- net ENRST: now also C32.1; no longer C32.2
- new net: D9.2 (A), R46.1
- new net: D8.1 (K), R45.2
- new net LGND: R45.1
- new net LVCC: R46.2
- new net SW_BOOT0: D8.2 (A), D9.1 (K), R44.1, SW5.2 (B)
Other:
- moved on the sheet: C28, C29, C30, C31, C32, C33, R41, R42, R43, SW4, U8
